Commit message: fix open_manipulator xacro
for consistency, does not effect actual urdf

File: ros2_ws/src/marvin/urdf/open_manipulator.urdf.xacro (robot description, xacro)
@@ -31,12 +31,12 @@
       <origin xyz="0 0 0" rpy="0 0 0"/>
       <geometry>
-        <mesh filename="install/marvin/share/marvin/urdf/meshes/chain_link1.stl" scale="0.001 0.001 0.001"/>
-      </geometry>
-      <material name="grey"/>
-    </visual>
-    <collision>
-      <origin xyz="0 0 0" rpy="0 0 0"/>
-      <geometry>
-        <mesh filename="install/marvin/share/marvin/urdf/meshes/chain_link1.stl" scale="0.001 0.001 0.001"/>
+        <mesh filename="package://marvin/urdf/meshes/chain_link1.stl" scale="0.001 0.001 0.001"/>
+      </geometry>
+      <material name="grey"/>
+    </visual>
+    <collision>
+      <origin xyz="0 0 0" rpy="0 0 0"/>
+      <geometry>
+        <mesh filename="package://marvin/urdf/meshes/chain_link1.stl" scale="0.001 0.001 0.001"/>
       </geometry>
     </collision>
@@ -62,5 +62,5 @@
       <origin xyz="0 0 0.019" rpy="0 0 0"/>
       <geometry>
-        <mesh filename="install/marvin/share/marvin/urdf/meshes/chain_link2.stl" scale="0.001 0.001 0.001"/>
+        <mesh filename="package://marvin/urdf/meshes/chain_link2.stl" scale="0.001 0.001 0.001"/>
       </geometry>
       <material name="grey"/>
@@ -69,5 +69,5 @@
       <origin xyz="0 0 0.019" rpy="0 0 0"/>
       <geometry>
-        <mesh filename="install/marvin/share/marvin/urdf/meshes/chain_link2.stl" scale="0.001 0.001 0.001"/>
+        <mesh filename="package://marvin/urdf/meshes/chain_link2.stl" scale="0.001 0.001 0.001"/>
       </geometry>
     </collision>
@@ -93,12 +93,12 @@
       <origin xyz="0 0 0" rpy="0 0 0"/>
       <geometry>
-        <mesh filename="install/marvin/share/marvin/urdf/meshes/chain_link3.stl" scale="0.001 0.001 0.001"/>
-      </geometry>
-      <material name="grey"/>
-    </visual>
-    <collision>
-      <origin xyz="0 0 0" rpy="0 0 0"/>
-      <geometry>
-        <mesh filename="install/marvin/share/marvin/urdf/meshes/chain_link3.stl" scale="0.001 0.001 0.001"/>
+        <mesh filename="package://marvin/urdf/meshes/chain_link3.stl" scale="0.001 0.001 0.001"/>
+      </geometry>
+      <material name="grey"/>
+    </visual>
+    <collision>
+      <origin xyz="0 0 0" rpy="0 0 0"/>
+      <geometry>
+        <mesh filename="package://marvin/urdf/meshes/chain_link3.stl" scale="0.001 0.001 0.001"/>
       </geometry>
     </collision>
@@ -124,12 +124,12 @@
       <origin xyz="0 0 0" rpy="0 0 0"/>
       <geometry>
-        <mesh filename="install/marvin/share/marvin/urdf/meshes/chain_link4.stl" scale="0.001 0.001 0.001"/>
-      </geometry>
-      <material name="grey"/>
-    </visual>
-    <collision>
-      <origin xyz="0 0 0" rpy="0 0 0"/>
-      <geometry>
-        <mesh filename="install/marvin/share/marvin/urdf/meshes/chain_link4.stl" scale="0.001 0.001 0.001"/>
+        <mesh filename="package://marvin/urdf/meshes/chain_link4.stl" scale="0.001 0.001 0.001"/>
+      </geometry>
+      <material name="grey"/>
+    </visual>
+    <collision>
+      <origin xyz="0 0 0" rpy="0 0 0"/>
+      <geometry>
+        <mesh filename="package://marvin/urdf/meshes/chain_link4.stl" scale="0.001 0.001 0.001"/>
       </geometry>
     </collision>
@@ -155,12 +155,12 @@
       <origin xyz="0 0 0" rpy="0 0 0"/>
       <geometry>
-        <mesh filename="install/marvin/share/marvin/urdf/meshes/chain_link5.stl" scale="0.001 0.001 0.001"/>
-      </geometry>
-      <material name="grey"/>
-    </visual>
-    <collision>
-      <origin xyz="0 0 0" rpy="0 0 0"/>
-      <geometry>
-        <mesh filename="install/marvin/share/marvin/urdf/meshes/chain_link5.stl" scale="0.001 0.001 0.001"/>
+        <mesh filename="package://marvin/urdf/meshes/chain_link5.stl" scale="0.001 0.001 0.001"/>
+      </geometry>
+      <material name="grey"/>
+    </visual>
+    <collision>
+      <origin xyz="0 0 0" rpy="0 0 0"/>
+      <geometry>
+        <mesh filename="package://marvin/urdf/meshes/chain_link5.stl" scale="0.001 0.001 0.001"/>
       </geometry>
     </collision>
@@ -186,5 +186,5 @@
       <origin xyz="0.0 0.0 0" rpy="0 0 0"/>
       <geometry>
-        <mesh filename="install/marvin/share/marvin/urdf/meshes/chain_link_grip_l.stl" scale="0.001 0.001 0.001"/>
+        <mesh filename="package://marvin/urdf/meshes/chain_link_grip_l.stl" scale="0.001 0.001 0.001"/>
       </geometry>
       <material name="grey"/>
@@ -193,5 +193,5 @@
       <origin xyz="0.0 0.0 0" rpy="0 0 0"/>
       <geometry>
-        <mesh filename="install/marvin/share/marvin/urdf/meshes/chain_link_grip_l.stl" scale="0.001 0.001 0.001"/>
+        <mesh filename="package://marvin/urdf/meshes/chain_link_grip_l.stl" scale="0.001 0.001 0.001"/>
       </geometry>
     </collision>
@@ -218,5 +218,5 @@
       <origin xyz="0.0 -0.0 0" rpy="0 0 0"/>
       <geometry>
-        <mesh filename="install/marvin/share/marvin/urdf/meshes/chain_link_grip_r.stl" scale="0.001 0.001 0.001"/>
+        <mesh filename="package://marvin/urdf/meshes/chain_link_grip_r.stl" scale="0.001 0.001 0.001"/>
       </geometry>
       <material name="grey"/>
@@ -225,5 +225,5 @@
       <origin xyz="0.0 -0.0 0" rpy="0 0 0"/>
       <geometry>
-        <mesh filename="install/marvin/share/marvin/urdf/meshes/chain_link_grip_r.stl" scale="0.001 0.001 0.001"/>
+        <mesh filename="package://marvin/urdf/meshes/chain_link_grip_r.stl" scale="0.001 0.001 0.001"/>
       </geometry>
     </collision>

Commit message: control joint1 with shoulder

File: ros2_ws/src/marvin/urdf/open_manipulator.urdf.xacro (robot description, xacro)
@@ -1,29 +1,19 @@
 <?xml version="1.0"?>
-<!-- Open_Manipulator Chain -->
-<robot xmlns:xacro="http://www.ros.org/wiki/xacro" name="open_manipulator">
-  <material name="black">
-    <color rgba="0.0 0.0 0.0 1.0"/>
-  </material>
-  <material name="white">
-    <color rgba="1.0 1.0 1.0 1.0"/>
-  </material>
+<robot name="open_manipulator" xmlns:xacro="http://www.ros.org/wiki/xacro">
   <material name="red">
     <color rgba="0.8 0.0 0.0 1.0"/>
-  </material>
-  <material name="blue">
-    <color rgba="0.0 0.0 0.8 1.0"/>
-  </material>
-  <material name="green">
-    <color rgba="0.0 0.8 0.0 1.0"/>
   </material>
   <material name="grey">
     <color rgba="0.5 0.5 0.5 1.0"/>
   </material>
-  <material name="orange">
-    <color rgba="1.0 0.4235294117647059 0.0392156862745098 1.0"/>
-  </material>
-  <material name="brown">
-    <color rgba="0.8705882352941177 0.8117647058823529 0.7647058823529411 1.0"/>
-  </material>
+  <!-- Dummy link as new root -->
+  <link name="dummy_link">
+  </link>
+  <!-- Dummy joint to connect the dummy link with the original base link -->
+  <joint name="dummy_joint" type="fixed">
+    <origin xyz="0 0 0" rpy="0 0 0"/>
+    <parent link="dummy_link"/>
+    <child link="base_link"/>
+  </joint>
   <!-- Link 1 -->
   <link name="base_link">

Commit message: Update README

File: ros2_ws/src/marvin/urdf/open_manipulator.urdf.xacro (robot description, xacro)
@@ -7,13 +7,4 @@
     <color rgba="0.5 0.5 0.5 1.0"/>
   </material>
-  <!-- Dummy link as new root -->
-  <link name="dummy_link">
-  </link>
-  <!-- Dummy joint to connect the dummy link with the original base link -->
-  <joint name="dummy_joint" type="fixed">
-    <origin xyz="0 0 0" rpy="0 0 0"/>
-    <parent link="dummy_link"/>
-    <child link="base_link"/>
-  </joint>
   <!-- Link 1 -->
   <link name="base_link">
