Commit message: urdf can be opend in rviz2

File: ros2_ws/src/marvin/urdf/marvin.urdf (robot description, URDF)
Before this commit: robot simple_two_armed_robot, 3 links, 2 joints
Links:
- removed link body
- added link base_link; visual box size=0.5 0.5 1
Joints:
- joint left_shoulder: axis 1 0 0 -> 0 1 0; limit lower=- upper=1 effort=100 velocity=0.5 -> lower=-1.5 upper=1.5 effort=100 velocity=0.5; origin xyz=0.25 0 -0.5 rpy=0 0 0 -> xyz=0.25 0 0.5 rpy=0 0 0; parent body -> base_link
- joint right_shoulder: axis 1 0 0 -> 0 1 0; limit lower=- upper=1 effort=100 velocity=0.5 -> lower=-1.5 upper=1.5 effort=100 velocity=0.5; origin xyz=-0.25 0 -0.5 rpy=0 0 0 -> xyz=-0.25 0 0.5 rpy=0 0 0; parent body -> base_link

File: ros2_ws/src/marvin/urdf/marvin.xacro (robot description, xacro)
@@ -2,5 +2,5 @@
 <robot xmlns:xacro="http://www.ros.org/wiki/xacro" name="simple_two_armed_robot">
   <!-- Macro Definitions -->
-  <xacro:macro name="cylinder_link" params="name length radius color">
+  <xacro:macro name="cylinder_link" params="name length radius origin color">
     <link name="${name}">
       <visual>
@@ -8,9 +8,10 @@
           <cylinder length="${length}" radius="${radius}"/>
         </geometry>
+        <origin xyz="${origin}" rpy="0 0 0"/>
         <material name="${color}"/>
       </visual>
     </link>
   </xacro:macro>
-  <xacro:macro name="revolute_joint" params="name parent child origin axis limit">
+  <xacro:macro name="revolute_joint" params="name parent child origin axis lower_limit upper_limit">
     <joint name="${name}" type="revolute">
       <parent link="${parent}"/>
@@ -18,5 +19,5 @@
       <origin xyz="${origin}" rpy="0 0 0"/>
       <axis xyz="${axis}"/>
-      <limit lower="${limit[0]}" upper="${limit[1]}" effort="100" velocity="0.5"/>
+      <limit lower="${lower_limit}" upper="${upper_limit}" effort="100" velocity="0.5"/>
     </joint>
   </xacro:macro>
@@ -31,6 +32,6 @@
     <color rgba="1 0 0 1"/>
   </material>
-  <!-- Body (Torso) Link -->
-  <link name="body">
+  <!-- base_link (Torso) Link -->
+  <link name="base_link">
     <visual>
       <geometry>
@@ -41,8 +42,8 @@
   </link>
   <!-- Left and Right Arm Links -->
-  <xacro:cylinder_link name="left_arm" length="1" radius="0.1" color="green"/>
-  <xacro:cylinder_link name="right_arm" length="1" radius="0.1" color="red"/>
+  <xacro:cylinder_link name="left_arm" length="1" radius="0.1" origin="0.1 0 -0.5" color="green"/>
+  <xacro:cylinder_link name="right_arm" length="1" radius="0.1" origin="-0.1 0 -0.5" color="red"/>
   <!-- Left and Right Shoulder Joints -->
-  <xacro:revolute_joint name="left_shoulder" parent="body" child="left_arm" origin="0.25 0 -0.5" axis="1 0 0" limit="-1.5 1.5"/>
-  <xacro:revolute_joint name="right_shoulder" parent="body" child="right_arm" origin="-0.25 0 -0.5" axis="1 0 0" limit="-1.5 1.5"/>
+  <xacro:revolute_joint name="left_shoulder" parent="base_link" child="left_arm" origin="0.25 0 0.5" axis="0 1 0" lower_limit="-1.5" upper_limit="1.5"/>
+  <xacro:revolute_joint name="right_shoulder" parent="base_link" child="right_arm" origin="-0.25 0 0.5" axis="0 1 0" lower_limit="-1.5" upper_limit="1.5"/>
 </robot>

Commit message: urdf with body

File: ros2_ws/src/marvin/urdf/marvin.urdf (robot description, URDF)
Before this commit: robot marvin, 16 links, 15 joints
Links:
- removed link world
- added link body; collision box size=0.16000 0.06000 0.60000
Joints:
- removed joint base_joint
- added joint marvin_to_body: type fixed, parent body, child marvin, origin xyz=0.00000 0.00000 0.00000 rpy=0.00000 0.00000 0.00000

Commit message: pre moveit package

File: ros2_ws/src/marvin/urdf/marvin.urdf (robot description, URDF)
Before this commit: robot marvin, 16 links, 15 joints
Links:
- removed link body
- removed link left_end_effector_link
- removed link left_gripper_link
- removed link left_gripper_link_sub
- removed link left_link2
- removed link left_link3
- removed link left_link4
- removed link left_link5
- removed link marvin
- removed link right_end_effector_link
- removed link right_gripper_link
- removed link right_gripper_link_sub
- removed link right_link2
- removed link right_link3
- removed link right_link4
- removed link right_link5
- added link end_effector_link, mass 1.0e-03; visual box size=0.01 0.01 0.01
- added link gripper_link, mass 1.0e-03; collision mesh filename=package://open_manipulator_description/meshes/chain_link_gr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 scale=0.001 0.001 0.001; visual mesh filename=package://open_manipulator_description/meshes/chain_link_gr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 scale=0.001 0.001 0.001
- added link gripper_link_sub, mass 1.0e-03; collision mesh filename=package://open_manipulator_description/meshes/chain_link_gr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 scale=0.001 0.001 0.001; visual mesh filename=package://open_manipulator_description/meshes/chain_link_gr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 scale=0.001 0.001 0.001
- added link link1, mass 7.9119962e-02; collision mesh filename=package://open_manipulator_description/meshes/chain_link1.s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 scale=0.001 0.001 0.001; visual mesh filename=package://open_manipulator_description/meshes/chain_link1.s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 scale=0.001 0.001 0.001
- added link link2, mass 9.8406837e-02; collision mesh filename=package://open_manipulator_description/meshes/chain_link2.s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 scale=0.001 0.001 0.001; visual mesh filename=package://open_manipulator_description/meshes/chain_link2.s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 scale=0.001 0.001 0.001
- added link link3, mass 1.3850917e-01; collision mesh filename=package://open_manipulator_description/meshes/chain_link3.s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 scale=0.001 0.001 0.001; visual mesh filename=package://open_manipulator_description/meshes/chain_link3.s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 scale=0.001 0.001 0.001
- added link link4, mass 1.3274562e-01; collision mesh filename=package://open_manipulator_description/meshes/chain_link4.s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 scale=0.001 0.001 0.001; visual mesh filename=package://open_manipulator_description/meshes/chain_link4.s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 scale=0.001 0.001 0.001
- added link link5, mass 1.4327573e-01; collision mesh filename=package://open_manipulator_description/meshes/chain_link5.s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 scale=0.001 0.001 0.001; visual mesh filename=package://open_manipulator_description/meshes/chain_link5.s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 scale=0.001 0.001 0.001
- added link torso; collision box size=0.16000 0.06000 0.60000
- added link world
Joints:
- removed joint left_end_effector_joint
- removed joint left_gripper
- removed joint left_gripper_sub
- removed joint left_joint1
- removed joint left_joint2
- removed joint left_joint3
- removed joint left_joint4
- removed joint marvin_to_body
- removed joint right_end_effector_joint
- removed joint right_gripper
- removed joint right_gripper_sub
- removed joint right_joint1
- removed joint right_joint2
- removed joint right_joint3
- removed joint right_joint4
- added joint end_effector_joint: type fixed, parent link5, child end_effector_link, origin xyz=0.126 0.0 0.0 rpy=0 0 0
- added joint gripper: type prismatic, parent link5, child gripper_link, origin xyz=0.0817 0.021 0.0 rpy=0 0 0, axis 0 1 0, limit lower=-0.010 upper=0.019 effort=1 velocity=4.8
- added joint gripper_sub: type prismatic, parent link5, child gripper_link_sub, origin xyz=0.0817 -0.021 0 rpy=0 0 0, axis 0 -1 0, limit lower=-0.010 upper=0.019 effort=1 velocity=4.8, mimic joint=gripper multiplier=1
- added joint joint1: type revolute, parent link1, child link2, origin xyz=0.012 0.0 0.017 rpy=0 0 0, axis 0 0 1, limit lower=-2.827433388230814 upper=2.827433388230814 effort=1 velocity=4.8
- added joint joint2: type revolute, parent link2, child link3, origin xyz=0.0 0.0 0.0595 rpy=0 0 0, axis 0 1 0, limit lower=-1.790707812546182 upper=1.5707963267948966 effort=1 velocity=4.8
- added joint joint3: type revolute, parent link3, child link4, origin xyz=0.024 0 0.128 rpy=0 0 0, axis 0 1 0, limit lower=-0.9424777960769379 upper=1.382300767579509 effort=1 velocity=4.8
- added joint joint4: type revolute, parent link4, child link5, origin xyz=0.124 0.0 0.0 rpy=0 0 0, axis 0 1 0, limit lower=-1.790707812546182 upper=2.0420352248333655 effort=1 velocity=4.8
- added joint left_arm_joint: type fixed, parent torso, child left_arm_base, origin xyz=0.5 0.2 0 rpy=0 0 0
- added joint right_arm_joint: type fixed, parent torso, child right_arm_base, origin xyz=-0.5 0.2 0 rpy=0 0 3.141592653589793
- added joint world_fixed: type fixed, parent world, child link1, origin xyz=0 0 0 rpy=0 0 0

File: ros2_ws/src/marvin_moveit/config/marvin.ros2_control.xacro (robot description, xacro)
@@ -2,5 +2,5 @@
 <robot xmlns:xacro="http://www.ros.org/wiki/xacro">
     <xacro:macro name="marvin_ros2_control" params="name initial_positions_file">
-        <xacro:property name="initial_positions" value="${load_yaml(initial_positions_file)['initial_positions']}"/>
+        <xacro:property name="initial_positions" value="${xacro.load_yaml(initial_positions_file)['initial_positions']}"/>
         <ros2_control name="${name}" type="system">
             <hardware>
@@ -14,4 +14,5 @@
                 </state_interface>
                 <state_interface name="velocity"/>
+                <state_interface name="effort"/>
             </joint>
             <joint name="right_joint2">
@@ -21,4 +22,5 @@
                 </state_interface>
                 <state_interface name="velocity"/>
+                <state_interface name="effort"/>
             </joint>
             <joint name="right_joint3">
@@ -28,4 +30,5 @@
                 </state_interface>
                 <state_interface name="velocity"/>
+                <state_interface name="effort"/>
             </joint>
             <joint name="right_joint4">
@@ -35,4 +38,5 @@
                 </state_interface>
                 <state_interface name="velocity"/>
+                <state_interface name="effort"/>
             </joint>
             <joint name="right_gripper">
@@ -42,4 +46,5 @@
                 </state_interface>
                 <state_interface name="velocity"/>
+                <state_interface name="effort"/>
             </joint>
             <joint name="left_joint1">
@@ -49,4 +54,5 @@
                 </state_interface>
                 <state_interface name="velocity"/>
+                <state_interface name="effort"/>
             </joint>
             <joint name="left_joint2">
@@ -56,4 +62,5 @@
                 </state_interface>
                 <state_interface name="velocity"/>
+                <state_interface name="effort"/>
             </joint>
             <joint name="left_joint3">
@@ -63,4 +70,5 @@
                 </state_interface>
                 <state_interface name="velocity"/>
+                <state_interface name="effort"/>
             </joint>
             <joint name="left_joint4">
@@ -70,4 +78,5 @@
                 </state_interface>
                 <state_interface name="velocity"/>
+                <state_interface name="effort"/>
             </joint>
             <joint name="left_gripper">
@@ -77,4 +86,5 @@
                 </state_interface>
                 <state_interface name="velocity"/>
+                <state_interface name="effort"/>
             </joint>
         </ros2_control>

Commit message: urdf two arms

File: ros2_ws/src/marvin/urdf/marvin.urdf (robot description, URDF)
Before this commit: robot marvin, 10 links, 10 joints
Links:
- link gripper_link: geometry collision mesh filename=../meshes/chain_link_grip_l.stl scale=0.001 0.001 0.001; visual mesh filename=../meshes/chain_link_grip_l.stl scale=0.001 0.001 0.001
- link gripper_link_sub: geometry collision mesh filename=../meshes/stl/chain_link_grip_r.stl scale=0.001 0.001 0.001; visual mesh filename=../meshes/chain_link_grip_r.stl scale=0.001 0.001 0.001
- link link1: geometry collision mesh filename=../meshes/chain_link1.stl scale=0.001 0.001 0.001; visual mesh filename=../meshes/chain_link1.stl scale=0.001 0.001 0.001
- link link2: geometry collision mesh filename=../meshes/chain_link2.stl scale=0.001 0.001 0.001; visual mesh filename=../meshes/chain_link2.stl scale=0.001 0.001 0.001
- link link3: geometry collision mesh filename=../meshes/chain_link3.stl scale=0.001 0.001 0.001; visual mesh filename=../meshes/chain_link3.stl scale=0.001 0.001 0.001
- link link4: geometry collision mesh filename=../meshes/chain_link4.stl scale=0.001 0.001 0.001; visual mesh filename=../meshes/chain_link4.stl scale=0.001 0.001 0.001
- link link5: geometry collision mesh filename=../meshes/chain_link5.stl scale=0.001 0.001 0.001; visual mesh filename=../meshes/chain_link5.stl scale=0.001 0.001 0.001
Joints:
- joint left_arm_joint: child left_arm_base -> link1
- joint right_arm_joint: child right_arm_base -> link1
- joint world_fixed: child link1 -> torso

File: ros2_ws/src/marvin/urdf2/marvin.urdf.xacro (robot description, xacro)
@@ -5,9 +5,10 @@
   <xacro:include filename="/home/jaeho/marvin/ros2_ws/src/marvin/urdf2/materials.xacro" />
   <!-- Import all Gazebo-customization elements, including Gazebo colors -->
-  <xacro:include filename="/home/jaeho/marvin/ros2_ws/src/marvin/urdf2/open_manipulator.gazebo.xacro" />
+  <!--xacro:include filename="/home/jaeho/marvin/ros2_ws/src/marvin/urdf2/open_manipulator.gazebo.xacro" /-->
   <!-- Import Transmission -->
   <xacro:include filename="/home/jaeho/marvin/ros2_ws/src/marvin/urdf2/open_manipulator.transmission.xacro" />
   <!-- Import URDF -->
-  <xacro:include filename="/home/jaeho/marvin/ros2_ws/src/marvin/urdf2/open_manipulator.urdf.xacro" />
+  <!--xacro:include filename="/home/jaeho/marvin/ros2_ws/src/marvin/urdf2/open_manipulator.urdf.xacro" /-->
+  <xacro:include filename="/home/jaeho/marvin/ros2_ws/src/marvin/urdf2/single_arm.xacro" />
   <!-- World -->
   <link name="world"/>
@@ -16,5 +17,5 @@
     <origin xyz="0 0 0" rpy="0 0 0"/>
     <parent link="world"/>
-    <child link="link1"/>
+    <child link="torso"/>
   </joint>
   <!-- Torso Link -->
@@ -26,19 +27,27 @@
       </geometry>
     </collision>
+    <visual name="Cube">
+      <origin rpy="0.00000 0.00000 0.00000" xyz="0.00000 0.00000 -0.22261"/>
+      <geometry>
+        <box size="0.16000 0.06000 0.60000"/>
+      </geometry>
+    </visual>
+    <parent link="world"/>
   </link>
-  <!-- Left Arm -->
-  <!--xacro:include filename="single_arm.xacro"/-->
-  <xacro:property name="left_arm_origin" value="0.5 0.2 0"/>
+  <xacro:property name="left_arm_origin_xyz" value="0.08 0 0"/>
   <joint name="left_arm_joint" type="fixed">
     <parent link="torso"/>
-    <child link="left_arm_base"/>
-    <origin xyz="${left_arm_origin}" rpy="0 0 0"/>
+    <child link="link1_left"/>
+    <origin xyz="${left_arm_origin_xyz}" rpy="0 1.5708 0"/>
   </joint>
-  <!-- Right Arm (mirrored) -->
-  <xacro:property name="right_arm_origin" value="-0.5 0.2 0"/>
+  <xacro:property name="right_arm_origin_xyz" value="-0.08 0 0"/>
   <joint name="right_arm_joint" type="fixed">
     <parent link="torso"/>
-    <child link="right_arm_base"/>
-    <origin xyz="${right_arm_origin}" rpy="0 0 ${pi}"/>
+    <child link="link1_right"/>
+    <origin xyz="${right_arm_origin_xyz}" rpy="0 1.5708 3.1415926535"/> <!-- Rotate by pi -->
   </joint>
+  <xacro:arm name="left"/>
+   <!-- Left Arm -->
+  <xacro:arm name="right"/>
+  <!-- Right Arm (Mirrored) -->
 </robot>

File: ros2_ws/src/marvin/urdf2/open_manipulator.urdf.xacro (robot description, xacro)
@@ -7,12 +7,12 @@
       <origin xyz="0 0 0" rpy="0 0 0"/>
       <geometry>
-        <mesh filename="package://open_manipulator_description/meshes/chain_link1.stl" scale="0.001 0.001 0.001"/>
-      </geometry>
-      <material name="grey"/>
-    </visual>
-    <collision>
-      <origin xyz="0 0 0" rpy="0 0 0"/>
-      <geometry>
-        <mesh filename="package://open_manipulator_description/meshes/chain_link1.stl" scale="0.001 0.001 0.001"/>
+        <mesh filename="../meshes/stl/chain_link1.stl" scale="0.001 0.001 0.001"/>
+      </geometry>
+      <material name="grey"/>
+    </visual>
+    <collision>
+      <origin xyz="0 0 0" rpy="0 0 0"/>
+      <geometry>
+        <mesh filename="../meshes/stl/chain_link1.stl" scale="0.001 0.001 0.001"/>
       </geometry>
     </collision>
@@ -38,5 +38,5 @@
       <origin xyz="0 0 0.019" rpy="0 0 0"/>
       <geometry>
-        <mesh filename="package://open_manipulator_description/meshes/chain_link2.stl" scale="0.001 0.001 0.001"/>
+        <mesh filename="../meshes/stl/chain_link2.stl" scale="0.001 0.001 0.001"/>
       </geometry>
       <material name="grey"/>
@@ -45,5 +45,5 @@
       <origin xyz="0 0 0.019" rpy="0 0 0"/>
       <geometry>
-        <mesh filename="package://open_manipulator_description/meshes/chain_link2.stl" scale="0.001 0.001 0.001"/>
+        <mesh filename="../meshes/stl/chain_link2.stl" scale="0.001 0.001 0.001"/>
       </geometry>
     </collision>
@@ -69,12 +69,12 @@
       <origin xyz="0 0 0" rpy="0 0 0"/>
       <geometry>
-        <mesh filename="package://open_manipulator_description/meshes/chain_link3.stl" scale="0.001 0.001 0.001"/>
-      </geometry>
-      <material name="grey"/>
-    </visual>
-    <collision>
-      <origin xyz="0 0 0" rpy="0 0 0"/>
-      <geometry>
-        <mesh filename="package://open_manipulator_description/meshes/chain_link3.stl" scale="0.001 0.001 0.001"/>
+        <mesh filename="../meshes/stl/chain_link3.stl" scale="0.001 0.001 0.001"/>
+      </geometry>
+      <material name="grey"/>
+    </visual>
+    <collision>
+      <origin xyz="0 0 0" rpy="0 0 0"/>
+      <geometry>
+        <mesh filename="../meshes/stl/chain_link3.stl" scale="0.001 0.001 0.001"/>
       </geometry>
     </collision>
@@ -100,12 +100,12 @@
       <origin xyz="0 0 0" rpy="0 0 0"/>
       <geometry>
-        <mesh filename="package://open_manipulator_description/meshes/chain_link4.stl" scale="0.001 0.001 0.001"/>
-      </geometry>
-      <material name="grey"/>
-    </visual>
-    <collision>
-      <origin xyz="0 0 0" rpy="0 0 0"/>
-      <geometry>
-        <mesh filename="package://open_manipulator_description/meshes/chain_link4.stl" scale="0.001 0.001 0.001"/>
+        <mesh filename="../meshes/stl/chain_link4.stl" scale="0.001 0.001 0.001"/>
+      </geometry>
+      <material name="grey"/>
+    </visual>
+    <collision>
+      <origin xyz="0 0 0" rpy="0 0 0"/>
+      <geometry>
+        <mesh filename="../meshes/stl/chain_link4.stl" scale="0.001 0.001 0.001"/>
       </geometry>
     </collision>
@@ -131,12 +131,12 @@
       <origin xyz="0 0 0" rpy="0 0 0"/>
       <geometry>
-        <mesh filename="package://open_manipulator_description/meshes/chain_link5.stl" scale="0.001 0.001 0.001"/>
-      </geometry>
-      <material name="grey"/>
-    </visual>
-    <collision>
-      <origin xyz="0 0 0" rpy="0 0 0"/>
-      <geometry>
-        <mesh filename="package://open_manipulator_description/meshes/chain_link5.stl" scale="0.001 0.001 0.001"/>
+        <mesh filename="../meshes/stl/chain_link5.stl" scale="0.001 0.001 0.001"/>
+      </geometry>
+      <material name="grey"/>
+    </visual>
+    <collision>
+      <origin xyz="0 0 0" rpy="0 0 0"/>
+      <geometry>
+        <mesh filename="../meshes/stl/chain_link5.stl" scale="0.001 0.001 0.001"/>
       </geometry>
     </collision>
@@ -162,5 +162,5 @@
       <origin xyz="0.0 0.0 0" rpy="0 0 0"/>
       <geometry>
-        <mesh filename="package://open_manipulator_description/meshes/chain_link_grip_l.stl" scale="0.001 0.001 0.001"/>
+        <mesh filename="../meshes/stl/chain_link_grip_l.stl" scale="0.001 0.001 0.001"/>
       </geometry>
       <material name="grey"/>
@@ -169,5 +169,5 @@
       <origin xyz="0.0 0.0 0" rpy="0 0 0"/>
       <geometry>
-        <mesh filename="package://open_manipulator_description/meshes/chain_link_grip_l.stl" scale="0.001 0.001 0.001"/>
+        <mesh filename="../meshes/stl/chain_link_grip_l.stl" scale="0.001 0.001 0.001"/>
       </geometry>
     </collision>
@@ -194,5 +194,5 @@
       <origin xyz="0.0 -0.0 0" rpy="0 0 0"/>
       <geometry>
-        <mesh filename="package://open_manipulator_description/meshes/chain_link_grip_r.stl" scale="0.001 0.001 0.001"/>
+        <mesh filename="../meshes/stl/chain_link_grip_r.stl" scale="0.001 0.001 0.001"/>
       </geometry>
       <material name="grey"/>
@@ -201,5 +201,5 @@
       <origin xyz="0.0 -0.0 0" rpy="0 0 0"/>
       <geometry>
-        <mesh filename="package://open_manipulator_description/meshes/chain_link_grip_r.stl" scale="0.001 0.001 0.001"/>
+        <mesh filename="../meshes/stl/chain_link_grip_r.stl" scale="0.001 0.001 0.001"/>
       </geometry>
     </collision>
