Commit message: move urdf2 to urdf

File: ros2_ws/src/marvin/urdf/marvin.urdf (robot description, URDF)
Before this commit: robot marvin, 10 links, 10 joints
Links:
- removed link end_effector_link
- removed link gripper_link
- removed link gripper_link_sub
- removed link link1
- removed link link2
- removed link link3
- removed link link4
- removed link link5
- added link end_effector_link_left, mass 1.0e-03; visual box size=0.01 0.01 0.01
- added link end_effector_link_right, mass 1.0e-03; visual box size=0.01 0.01 0.01
- added link gripper_link_left, mass 1.0e-03; collision mesh filename=/home/jaeho/marvin/ros2_ws/install/marvin/share/marvin/mesh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 scale=0.001 0.001 0.001; visual mesh filename=/home/jaeho/marvin/ros2_ws/install/marvin/share/marvin/mesh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 scale=0.001 0.001 0.001
- added link gripper_link_right, mass 1.0e-03; collision mesh filename=/home/jaeho/marvin/ros2_ws/install/marvin/share/marvin/mesh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 scale=0.001 0.001 0.001; visual mesh filename=/home/jaeho/marvin/ros2_ws/install/marvin/share/marvin/mesh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 scale=0.001 0.001 0.001
- added link gripper_link_sub_left, mass 1.0e-03; collision mesh filename=/home/jaeho/marvin/ros2_ws/install/marvin/share/marvin/mesh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 scale=0.001 0.001 0.001; visual mesh filename=/home/jaeho/marvin/ros2_ws/install/marvin/share/marvin/mesh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 scale=0.001 0.001 0.001
- added link gripper_link_sub_right, mass 1.0e-03; collision mesh filename=/home/jaeho/marvin/ros2_ws/install/marvin/share/marvin/mesh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 scale=0.001 0.001 0.001; visual mesh filename=/home/jaeho/marvin/ros2_ws/install/marvin/share/marvin/mesh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 scale=0.001 0.001 0.001
- added link link1_left, mass 7.9119962e-02; collision mesh filename=/home/jaeho/marvin/ros2_ws/install/marvin/share/marvin/mesh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 scale=0.001 0.001 0.001; visual mesh filename=/home/jaeho/marvin/ros2_ws/install/marvin/share/marvin/mesh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 scale=0.001 0.001 0.001
- added link link1_right, mass 7.9119962e-02; collision mesh filename=/home/jaeho/marvin/ros2_ws/install/marvin/share/marvin/mesh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 scale=0.001 0.001 0.001; visual mesh filename=/home/jaeho/marvin/ros2_ws/install/marvin/share/marvin/mesh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 scale=0.001 0.001 0.001
- added link link2_left, mass 9.8406837e-02; collision mesh filename=/home/jaeho/marvin/ros2_ws/install/marvin/share/marvin/mesh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 scale=0.001 0.001 0.001; visual mesh filename=/home/jaeho/marvin/ros2_ws/install/marvin/share/marvin/mesh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 scale=0.001 0.001 0.001
- added link link2_right, mass 9.8406837e-02; collision mesh filename=/home/jaeho/marvin/ros2_ws/install/marvin/share/marvin/mesh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 scale=0.001 0.001 0.001; visual mesh filename=/home/jaeho/marvin/ros2_ws/install/marvin/share/marvin/mesh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 scale=0.001 0.001 0.001
- added link link3_left, mass 1.3850917e-01; collision mesh filename=/home/jaeho/marvin/ros2_ws/install/marvin/share/marvin/mesh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 scale=0.001 0.001 0.001; visual mesh filename=/home/jaeho/marvin/ros2_ws/install/marvin/share/marvin/mesh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 scale=0.001 0.001 0.001
- added link link3_right, mass 1.3850917e-01; collision mesh filename=/home/jaeho/marvin/ros2_ws/install/marvin/share/marvin/mesh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 scale=0.001 0.001 0.001; visual mesh filename=/home/jaeho/marvin/ros2_ws/install/marvin/share/marvin/mesh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 scale=0.001 0.001 0.001
- added link link4_left, mass 1.3274562e-01; collision mesh filename=/home/jaeho/marvin/ros2_ws/install/marvin/share/marvin/mesh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 scale=0.001 0.001 0.001; visual mesh filename=/home/jaeho/marvin/ros2_ws/install/marvin/share/marvin/mesh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 scale=0.001 0.001 0.001
- added link link4_right, mass 1.3274562e-01; collision mesh filename=/home/jaeho/marvin/ros2_ws/install/marvin/share/marvin/mesh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 scale=0.001 0.001 0.001; visual mesh filename=/home/jaeho/marvin/ros2_ws/install/marvin/share/marvin/mesh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 scale=0.001 0.001 0.001
- added link link5_left, mass 1.4327573e-01; collision mesh filename=/home/jaeho/marvin/ros2_ws/install/marvin/share/marvin/mesh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 scale=0.001 0.001 0.001; visual mesh filename=/home/jaeho/marvin/ros2_ws/install/marvin/share/marvin/mesh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 scale=0.001 0.001 0.001
- added link link5_right, mass 1.4327573e-01; collision mesh filename=/home/jaeho/marvin/ros2_ws/install/marvin/share/marvin/mesh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 scale=0.001 0.001 0.001; visual mesh filename=/home/jaeho/marvin/ros2_ws/install/marvin/share/marvin/mesh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 scale=0.001 0.001 0.001
- link torso: geometry collision box size=0.16000 0.06000 0.60000; visual box size=0.16000 0.06000 0.60000
Joints:
- removed joint end_effector_joint
- removed joint gripper
- removed joint gripper_sub
- removed joint joint1
- removed joint joint2
- removed joint joint3
- removed joint joint4
- added joint end_effector_joint_left: type fixed, parent link5_left, child end_effector_link_left, origin xyz=0.126 0.0 0.0 rpy=0 0 0
- added joint end_effector_joint_right: type fixed, parent link5_right, child end_effector_link_right, origin xyz=0.126 0.0 0.0 rpy=0 0 0
- added joint gripper_left: type prismatic, parent link5_left, child gripper_link_left, origin xyz=0.0817 0.021 0.0 rpy=0 0 0, axis 0 1 0, limit lower=-0.010 upper=0.019 effort=1 velocity=4.8
- added joint gripper_right: type prismatic, parent link5_right, child gripper_link_right, origin xyz=0.0817 0.021 0.0 rpy=0 0 0, axis 0 1 0, limit lower=-0.010 upper=0.019 effort=1 velocity=4.8
- added joint gripper_sub_left: type prismatic, parent link5_left, child gripper_link_sub_left, origin xyz=0.0817 -0.021 0 rpy=0 0 0, axis 0 -1 0, limit lower=-0.010 upper=0.019 effort=1 velocity=4.8, mimic joint=gripper_left multiplier=1
- added joint gripper_sub_right: type prismatic, parent link5_right, child gripper_link_sub_right, origin xyz=0.0817 -0.021 0 rpy=0 0 0, axis 0 -1 0, limit lower=-0.010 upper=0.019 effort=1 velocity=4.8, mimic joint=gripper_right multiplier=1
- added joint joint1_left: type revolute, parent link1_left, child link2_left, origin xyz=0.012 0.0 0.017 rpy=0 0 0, axis 0 0 1, limit lower=-2.827433388230814 upper=2.827433388230814 effort=1 velocity=4.8
- added joint joint1_right: type revolute, parent link1_right, child link2_right, origin xyz=0.012 0.0 0.017 rpy=0 0 0, axis 0 0 1, limit lower=-2.827433388230814 upper=2.827433388230814 effort=1 velocity=4.8
- added joint joint2_left: type revolute, parent link2_left, child link3_left, origin xyz=0.0 0.0 0.0595 rpy=0 0 0, axis 0 1 0, limit lower=-1.790707812546182 upper=1.5707963267948966 effort=1 velocity=4.8
- added joint joint2_right: type revolute, parent link2_right, child link3_right, origin xyz=0.0 0.0 0.0595 rpy=0 0 0, axis 0 1 0, limit lower=-1.790707812546182 upper=1.5707963267948966 effort=1 velocity=4.8
- added joint joint3_left: type revolute, parent link3_left, child link4_left, origin xyz=0.024 0 0.128 rpy=0 0 0, axis 0 1 0, limit lower=-0.9424777960769379 upper=1.382300767579509 effort=1 velocity=4.8
- added joint joint3_right: type revolute, parent link3_right, child link4_right, origin xyz=0.024 0 0.128 rpy=0 0 0, axis 0 1 0, limit lower=-0.9424777960769379 upper=1.382300767579509 effort=1 velocity=4.8
- added joint joint4_left: type revolute, parent link4_left, child link5_left, origin xyz=0.124 0.0 0.0 rpy=0 0 0, axis 0 1 0, limit lower=-1.790707812546182 upper=2.0420352248333655 effort=1 velocity=4.8
- added joint joint4_right: type revolute, parent link4_right, child link5_right, origin xyz=0.124 0.0 0.0 rpy=0 0 0, axis 0 1 0, limit lower=-1.790707812546182 upper=2.0420352248333655 effort=1 velocity=4.8
- joint left_arm_joint: child link1 -> link1_left; origin xyz=0.5 0.2 0 rpy=0 0 0 -> xyz=0.08 0 0 rpy=0 1.5708 0
- joint right_arm_joint: child link1 -> link1_right; origin xyz=-0.5 0.2 0 rpy=0 0 3.141592653589793 -> xyz=-0.08 0 0 rpy=0 1.5708 3.1415926535

File: ros2_ws/src/marvin/urdf/single_arm.xacro (robot description, xacro)
@@ -7,12 +7,12 @@
         <origin xyz="0 0 0" rpy="0 0 0"/>
         <geometry>
-          <mesh filename="../meshes/stl/chain_link1.stl" scale="0.001 0.001 0.001"/>
-        </geometry>
-        <material name="grey"/>
-      </visual>
-      <collision>
-        <origin xyz="0 0 0" rpy="0 0 0"/>
-        <geometry>
-          <mesh filename="../meshes/stl/chain_link1.stl" scale="0.001 0.001 0.001"/>
+          <mesh filename="$(find marvin)/meshes/stl/chain_link1.stl" scale="0.001 0.001 0.001"/>
+        </geometry>
+        <material name="grey"/>
+      </visual>
+      <collision>
+        <origin xyz="0 0 0" rpy="0 0 0"/>
+        <geometry>
+          <mesh filename="$(find marvin)/meshes/stl/chain_link1.stl" scale="0.001 0.001 0.001"/>
         </geometry>
       </collision>
@@ -39,5 +39,5 @@
         <origin xyz="0 0 0.019" rpy="0 0 0"/>
         <geometry>
-          <mesh filename="../meshes/stl/chain_link2.stl" scale="0.001 0.001 0.001"/>
+          <mesh filename="$(find marvin)/meshes/stl/chain_link2.stl" scale="0.001 0.001 0.001"/>
         </geometry>
         <material name="grey"/>
@@ -46,5 +46,5 @@
         <origin xyz="0 0 0.019" rpy="0 0 0"/>
         <geometry>
-          <mesh filename="../meshes/stl/chain_link2.stl" scale="0.001 0.001 0.001"/>
+          <mesh filename="$(find marvin)/meshes/stl/chain_link2.stl" scale="0.001 0.001 0.001"/>
         </geometry>
       </collision>
@@ -70,12 +70,12 @@
         <origin xyz="0 0 0" rpy="0 0 0"/>
         <geometry>
-          <mesh filename="../meshes/stl/chain_link3.stl" scale="0.001 0.001 0.001"/>
-        </geometry>
-        <material name="grey"/>
-      </visual>
-      <collision>
-        <origin xyz="0 0 0" rpy="0 0 0"/>
-        <geometry>
-          <mesh filename="../meshes/stl/chain_link3.stl" scale="0.001 0.001 0.001"/>
+          <mesh filename="$(find marvin)/meshes/stl/chain_link3.stl" scale="0.001 0.001 0.001"/>
+        </geometry>
+        <material name="grey"/>
+      </visual>
+      <collision>
+        <origin xyz="0 0 0" rpy="0 0 0"/>
+        <geometry>
+          <mesh filename="$(find marvin)/meshes/stl/chain_link3.stl" scale="0.001 0.001 0.001"/>
         </geometry>
       </collision>
@@ -101,12 +101,12 @@
         <origin xyz="0 0 0" rpy="0 0 0"/>
         <geometry>
-          <mesh filename="../meshes/stl/chain_link4.stl" scale="0.001 0.001 0.001"/>
-        </geometry>
-        <material name="grey"/>
-      </visual>
-      <collision>
-        <origin xyz="0 0 0" rpy="0 0 0"/>
-        <geometry>
-          <mesh filename="../meshes/stl/chain_link4.stl" scale="0.001 0.001 0.001"/>
+          <mesh filename="$(find marvin)/meshes/stl/chain_link4.stl" scale="0.001 0.001 0.001"/>
+        </geometry>
+        <material name="grey"/>
+      </visual>
+      <collision>
+        <origin xyz="0 0 0" rpy="0 0 0"/>
+        <geometry>
+          <mesh filename="$(find marvin)/meshes/stl/chain_link4.stl" scale="0.001 0.001 0.001"/>
         </geometry>
       </collision>
@@ -132,12 +132,12 @@
         <origin xyz="0 0 0" rpy="0 0 0"/>
         <geometry>
-          <mesh filename="../meshes/stl/chain_link5.stl" scale="0.001 0.001 0.001"/>
-        </geometry>
-        <material name="grey"/>
-      </visual>
-      <collision>
-        <origin xyz="0 0 0" rpy="0 0 0"/>
-        <geometry>
-          <mesh filename="../meshes/stl/chain_link5.stl" scale="0.001 0.001 0.001"/>
+          <mesh filename="$(find marvin)/meshes/stl/chain_link5.stl" scale="0.001 0.001 0.001"/>
+        </geometry>
+        <material name="grey"/>
+      </visual>
+      <collision>
+        <origin xyz="0 0 0" rpy="0 0 0"/>
+        <geometry>
+          <mesh filename="$(find marvin)/meshes/stl/chain_link5.stl" scale="0.001 0.001 0.001"/>
         </geometry>
       </collision>
@@ -163,5 +163,5 @@
         <origin xyz="0.0 0.0 0" rpy="0 0 0"/>
         <geometry>
-          <mesh filename="../meshes/stl/chain_link_grip_l.stl" scale="0.001 0.001 0.001"/>
+          <mesh filename="$(find marvin)/meshes/stl/chain_link_grip_l.stl" scale="0.001 0.001 0.001"/>
         </geometry>
         <material name="grey"/>
@@ -170,5 +170,5 @@
         <origin xyz="0.0 0.0 0" rpy="0 0 0"/>
         <geometry>
-          <mesh filename="../meshes/stl/chain_link_grip_l.stl" scale="0.001 0.001 0.001"/>
+          <mesh filename="$(find marvin)/meshes/stl/chain_link_grip_l.stl" scale="0.001 0.001 0.001"/>
         </geometry>
       </collision>
@@ -195,5 +195,5 @@
         <origin xyz="0.0 -0.0 0" rpy="0 0 0"/>
         <geometry>
-          <mesh filename="../meshes/stl/chain_link_grip_r.stl" scale="0.001 0.001 0.001"/>
+          <mesh filename="$(find marvin)/meshes/stl/chain_link_grip_r.stl" scale="0.001 0.001 0.001"/>
         </geometry>
         <material name="grey"/>
@@ -202,5 +202,5 @@
         <origin xyz="0.0 -0.0 0" rpy="0 0 0"/>
         <geometry>
-          <mesh filename="../meshes/stl/chain_link_grip_r.stl" scale="0.001 0.001 0.001"/>
+          <mesh filename="$(find marvin)/meshes/stl/chain_link_grip_r.stl" scale="0.001 0.001 0.001"/>
         </geometry>
       </collision>

Commit message: marvin moveit

File: ros2_ws/src/marvin/urdf/marvin.urdf (robot description, URDF)
Before this commit: robot marvin, 18 links, 17 joints
Links:
- link gripper_link_left: geometry collision mesh filename=package://marvin/meshes/stl/chain_link_grip_l.stl scale=0.001 0.001 0.001; visual mesh filename=package://marvin/meshes/stl/chain_link_grip_l.stl scale=0.001 0.001 0.001
- link gripper_link_right: geometry collision mesh filename=package://marvin/meshes/stl/chain_link_grip_l.stl scale=0.001 0.001 0.001; visual mesh filename=package://marvin/meshes/stl/chain_link_grip_l.stl scale=0.001 0.001 0.001
- link gripper_link_sub_left: geometry collision mesh filename=package://marvin/meshes/stl/chain_link_grip_r.stl scale=0.001 0.001 0.001; visual mesh filename=package://marvin/meshes/stl/chain_link_grip_r.stl scale=0.001 0.001 0.001
- link gripper_link_sub_right: geometry collision mesh filename=package://marvin/meshes/stl/chain_link_grip_r.stl scale=0.001 0.001 0.001; visual mesh filename=package://marvin/meshes/stl/chain_link_grip_r.stl scale=0.001 0.001 0.001
- link link1_left: geometry collision mesh filename=package://marvin/meshes/stl/chain_link1.stl scale=0.001 0.001 0.001; visual mesh filename=package://marvin/meshes/stl/chain_link1.stl scale=0.001 0.001 0.001
- link link1_right: geometry collision mesh filename=package://marvin/meshes/stl/chain_link1.stl scale=0.001 0.001 0.001; visual mesh filename=package://marvin/meshes/stl/chain_link1.stl scale=0.001 0.001 0.001
- link link2_left: geometry collision mesh filename=package://marvin/meshes/stl/chain_link2.stl scale=0.001 0.001 0.001; visual mesh filename=package://marvin/meshes/stl/chain_link2.stl scale=0.001 0.001 0.001
- link link2_right: geometry collision mesh filename=package://marvin/meshes/stl/chain_link2.stl scale=0.001 0.001 0.001; visual mesh filename=package://marvin/meshes/stl/chain_link2.stl scale=0.001 0.001 0.001
- link link3_left: geometry collision mesh filename=package://marvin/meshes/stl/chain_link3.stl scale=0.001 0.001 0.001; visual mesh filename=package://marvin/meshes/stl/chain_link3.stl scale=0.001 0.001 0.001
- link link3_right: geometry collision mesh filename=package://marvin/meshes/stl/chain_link3.stl scale=0.001 0.001 0.001; visual mesh filename=package://marvin/meshes/stl/chain_link3.stl scale=0.001 0.001 0.001
- link link4_left: geometry collision mesh filename=package://marvin/meshes/stl/chain_link4.stl scale=0.001 0.001 0.001; visual mesh filename=package://marvin/meshes/stl/chain_link4.stl scale=0.001 0.001 0.001
- link link4_right: geometry collision mesh filename=package://marvin/meshes/stl/chain_link4.stl scale=0.001 0.001 0.001; visual mesh filename=package://marvin/meshes/stl/chain_link4.stl scale=0.001 0.001 0.001
- link link5_left: geometry collision mesh filename=package://marvin/meshes/stl/chain_link5.stl scale=0.001 0.001 0.001; visual mesh filename=package://marvin/meshes/stl/chain_link5.stl scale=0.001 0.001 0.001
- link link5_right: geometry collision mesh filename=package://marvin/meshes/stl/chain_link5.stl scale=0.001 0.001 0.001; visual mesh filename=package://marvin/meshes/stl/chain_link5.stl scale=0.001 0.001 0.001

File: ros2_ws/src/marvin_moveit/config/marvin.ros2_control.xacro (robot description, xacro)
@@ -8,83 +8,73 @@
                 <plugin>mock_components/GenericSystem</plugin>
             </hardware>
-            <joint name="right_joint1">
+            <joint name="joint1_left">
                 <command_interface name="position"/>
                 <state_interface name="position">
-                  <param name="initial_value">${initial_positions['right_joint1']}</param>
+                  <param name="initial_value">${initial_positions['joint1_left']}</param>
                 </state_interface>
                 <state_interface name="velocity"/>
-                <state_interface name="effort"/>
             </joint>
-            <joint name="right_joint2">
+            <joint name="joint2_left">
                 <command_interface name="position"/>
                 <state_interface name="position">
-                  <param name="initial_value">${initial_positions['right_joint2']}</param>
+                  <param name="initial_value">${initial_positions['joint2_left']}</param>
                 </state_interface>
                 <state_interface name="velocity"/>
-                <state_interface name="effort"/>
             </joint>
-            <joint name="right_joint3">
+            <joint name="joint3_left">
                 <command_interface name="position"/>
                 <state_interface name="position">
-                  <param name="initial_value">${initial_positions['right_joint3']}</param>
+                  <param name="initial_value">${initial_positions['joint3_left']}</param>
                 </state_interface>
                 <state_interface name="velocity"/>
-                <state_interface name="effort"/>
             </joint>
-            <joint name="right_joint4">
+            <joint name="joint4_left">
                 <command_interface name="position"/>
                 <state_interface name="position">
-                  <param name="initial_value">${initial_positions['right_joint4']}</param>
+                  <param name="initial_value">${initial_positions['joint4_left']}</param>
                 </state_interface>
                 <state_interface name="velocity"/>
-                <state_interface name="effort"/>
             </joint>
-            <joint name="right_gripper">
+            <joint name="joint1_right">
                 <command_interface name="position"/>
                 <state_interface name="position">
-                  <param name="initial_value">${initial_positions['right_gripper']}</param>
+                  <param name="initial_value">${initial_positions['joint1_right']}</param>
                 </state_interface>
                 <state_interface name="velocity"/>
-                <state_interface name="effort"/>
             </joint>
-            <joint name="left_joint1">
+            <joint name="joint2_right">
                 <command_interface name="position"/>
                 <state_interface name="position">
-                  <param name="initial_value">${initial_positions['left_joint1']}</param>
+                  <param name="initial_value">${initial_positions['joint2_right']}</param>
                 </state_interface>
                 <state_interface name="velocity"/>
-                <state_interface name="effort"/>
             </joint>
-            <joint name="left_joint2">
+            <joint name="joint3_right">
                 <command_interface name="position"/>
                 <state_interface name="position">
-                  <param name="initial_value">${initial_positions['left_joint2']}</param>
+                  <param name="initial_value">${initial_positions['joint3_right']}</param>
                 </state_interface>
                 <state_interface name="velocity"/>
-                <state_interface name="effort"/>
             </joint>
-            <joint name="left_joint3">
+            <joint name="joint4_right">
                 <command_interface name="position"/>
                 <state_interface name="position">
-                  <param name="initial_value">${initial_positions['left_joint3']}</param>
+                  <param name="initial_value">${initial_positions['joint4_right']}</param>
                 </state_interface>
                 <state_interface name="velocity"/>
-                <state_interface name="effort"/>
             </joint>
-            <joint name="left_joint4">
+            <joint name="gripper_left">
                 <command_interface name="position"/>
                 <state_interface name="position">
-                  <param name="initial_value">${initial_positions['left_joint4']}</param>
+                  <param name="initial_value">${initial_positions['gripper_left']}</param>
                 </state_interface>
                 <state_interface name="velocity"/>
-                <state_interface name="effort"/>
             </joint>
-            <joint name="left_gripper">
+            <joint name="gripper_right">
                 <command_interface name="position"/>
                 <state_interface name="position">
-                  <param name="initial_value">${initial_positions['left_gripper']}</param>
+                  <param name="initial_value">${initial_positions['gripper_right']}</param>
                 </state_interface>
                 <state_interface name="velocity"/>
-                <state_interface name="effort"/>
             </joint>
         </ros2_control>
