Commit message: joint velocity command publisher untested

File: ros2_ws/src/marvin/urdf/marvin.urdf (robot description, URDF)
Before this commit: robot marvin, 18 links, 17 joints
Links:
- removed link end_effector_link_left
- removed link end_effector_link_right
- removed link gripper_link_left
- removed link gripper_link_right
- removed link gripper_link_sub_left
- removed link gripper_link_sub_right
- removed link link1_left
- removed link link1_right
- removed link link2_left
- removed link link2_right
- removed link link3_left
- removed link link3_right
- removed link link4_left
- removed link link4_right
- removed link link5_left
- removed link link5_right
- added link left_end_effector_link, mass 1.0e-03; visual box size=0.01 0.01 0.01
- added link left_gripper_link, mass 1.0e-03; collision mesh filename=package://marvin/meshes/stl/chain_link_grip_l.stl scale=0.001 0.001 0.001; visual mesh filename=package://marvin/meshes/stl/chain_link_grip_l.stl scale=0.001 0.001 0.001
- added link left_gripper_link_sub, mass 1.0e-03; collision mesh filename=package://marvin/meshes/stl/chain_link_grip_r.stl scale=0.001 0.001 0.001; visual mesh filename=package://marvin/meshes/stl/chain_link_grip_r.stl scale=0.001 0.001 0.001
- added link left_link1, mass 7.9119962e-02; collision mesh filename=package://marvin/meshes/stl/chain_link1.stl scale=0.001 0.001 0.001; visual mesh filename=package://marvin/meshes/stl/chain_link1.stl scale=0.001 0.001 0.001
- added link left_link2, mass 9.8406837e-02; collision mesh filename=package://marvin/meshes/stl/chain_link2.stl scale=0.001 0.001 0.001; visual mesh filename=package://marvin/meshes/stl/chain_link2.stl scale=0.001 0.001 0.001
- added link left_link3, mass 1.3850917e-01; collision mesh filename=package://marvin/meshes/stl/chain_link3.stl scale=0.001 0.001 0.001; visual mesh filename=package://marvin/meshes/stl/chain_link3.stl scale=0.001 0.001 0.001
- added link left_link4, mass 1.3274562e-01; collision mesh filename=package://marvin/meshes/stl/chain_link4.stl scale=0.001 0.001 0.001; visual mesh filename=package://marvin/meshes/stl/chain_link4.stl scale=0.001 0.001 0.001
- added link left_link5, mass 1.4327573e-01; collision mesh filename=package://marvin/meshes/stl/chain_link5.stl scale=0.001 0.001 0.001; visual mesh filename=package://marvin/meshes/stl/chain_link5.stl scale=0.001 0.001 0.001
- added link right_end_effector_link, mass 1.0e-03; visual box size=0.01 0.01 0.01
- added link right_gripper_link, mass 1.0e-03; collision mesh filename=package://marvin/meshes/stl/chain_link_grip_l.stl scale=0.001 0.001 0.001; visual mesh filename=package://marvin/meshes/stl/chain_link_grip_l.stl scale=0.001 0.001 0.001
- added link right_gripper_link_sub, mass 1.0e-03; collision mesh filename=package://marvin/meshes/stl/chain_link_grip_r.stl scale=0.001 0.001 0.001; visual mesh filename=package://marvin/meshes/stl/chain_link_grip_r.stl scale=0.001 0.001 0.001
- added link right_link1, mass 7.9119962e-02; collision mesh filename=package://marvin/meshes/stl/chain_link1.stl scale=0.001 0.001 0.001; visual mesh filename=package://marvin/meshes/stl/chain_link1.stl scale=0.001 0.001 0.001
- added link right_link2, mass 9.8406837e-02; collision mesh filename=package://marvin/meshes/stl/chain_link2.stl scale=0.001 0.001 0.001; visual mesh filename=package://marvin/meshes/stl/chain_link2.stl scale=0.001 0.001 0.001
- added link right_link3, mass 1.3850917e-01; collision mesh filename=package://marvin/meshes/stl/chain_link3.stl scale=0.001 0.001 0.001; visual mesh filename=package://marvin/meshes/stl/chain_link3.stl scale=0.001 0.001 0.001
- added link right_link4, mass 1.3274562e-01; collision mesh filename=package://marvin/meshes/stl/chain_link4.stl scale=0.001 0.001 0.001; visual mesh filename=package://marvin/meshes/stl/chain_link4.stl scale=0.001 0.001 0.001
- added link right_link5, mass 1.4327573e-01; collision mesh filename=package://marvin/meshes/stl/chain_link5.stl scale=0.001 0.001 0.001; visual mesh filename=package://marvin/meshes/stl/chain_link5.stl scale=0.001 0.001 0.001
Joints:
- removed joint end_effector_joint_left
- removed joint end_effector_joint_right
- removed joint gripper_left
- removed joint gripper_right
- removed joint gripper_sub_left
- removed joint gripper_sub_right
- removed joint joint1_left
- removed joint joint1_right
- removed joint joint2_left
- removed joint joint2_right
- removed joint joint3_left
- removed joint joint3_right
- removed joint joint4_left
- removed joint joint4_right
- added joint left_end_effector_joint: type fixed, parent left_link5, child left_end_effector_link, origin xyz=0.126 0.0 0.0 rpy=0 0 0
- added joint left_gripper: type prismatic, parent left_link5, child left_gripper_link, origin xyz=0.0817 0.021 0.0 rpy=0 0 0, axis 0 1 0, limit lower=-0.010 upper=0.019 effort=1 velocity=4.8
- added joint left_gripper_sub: type prismatic, parent left_link5, child left_gripper_link_sub, origin xyz=0.0817 -0.021 0 rpy=0 0 0, axis 0 -1 0, limit lower=-0.010 upper=0.019 effort=1 velocity=4.8, mimic joint=left_gripper multiplier=1
- added joint left_joint1: type revolute, parent left_link1, child left_link2, origin xyz=0.012 0.0 0.017 rpy=0 0 0, axis 0 0 1, limit lower=-2.827433388230814 upper=2.827433388230814 effort=1 velocity=4.8
- added joint left_joint2: type revolute, parent left_link2, child left_link3, origin xyz=0.0 0.0 0.0595 rpy=0 0 0, axis 0 1 0, limit lower=-1.790707812546182 upper=1.5707963267948966 effort=1 velocity=4.8
- added joint left_joint3: type revolute, parent left_link3, child left_link4, origin xyz=0.024 0 0.128 rpy=0 0 0, axis 0 1 0, limit lower=-0.9424777960769379 upper=1.382300767579509 effort=1 velocity=4.8
- added joint left_joint4: type revolute, parent left_link4, child left_link5, origin xyz=0.124 0.0 0.0 rpy=0 0 0, axis 0 1 0, limit lower=-1.790707812546182 upper=2.0420352248333655 effort=1 velocity=4.8
- added joint right_end_effector_joint: type fixed, parent right_link5, child right_end_effector_link, origin xyz=0.126 0.0 0.0 rpy=0 0 0
- added joint right_gripper: type prismatic, parent right_link5, child right_gripper_link, origin xyz=0.0817 0.021 0.0 rpy=0 0 0, axis 0 1 0, limit lower=-0.010 upper=0.019 effort=1 velocity=4.8
- added joint right_gripper_sub: type prismatic, parent right_link5, child right_gripper_link_sub, origin xyz=0.0817 -0.021 0 rpy=0 0 0, axis 0 -1 0, limit lower=-0.010 upper=0.019 effort=1 velocity=4.8, mimic joint=right_gripper multiplier=1
- added joint right_joint1: type revolute, parent right_link1, child right_link2, origin xyz=0.012 0.0 0.017 rpy=0 0 0, axis 0 0 1, limit lower=-2.827433388230814 upper=2.827433388230814 effort=1 velocity=4.8
- added joint right_joint2: type revolute, parent right_link2, child right_link3, origin xyz=0.0 0.0 0.0595 rpy=0 0 0, axis 0 1 0, limit lower=-1.790707812546182 upper=1.5707963267948966 effort=1 velocity=4.8
- added joint right_joint3: type revolute, parent right_link3, child right_link4, origin xyz=0.024 0 0.128 rpy=0 0 0, axis 0 1 0, limit lower=-0.9424777960769379 upper=1.382300767579509 effort=1 velocity=4.8
- added joint right_joint4: type revolute, parent right_link4, child right_link5, origin xyz=0.124 0.0 0.0 rpy=0 0 0, axis 0 1 0, limit lower=-1.790707812546182 upper=2.0420352248333655 effort=1 velocity=4.8
- joint left_arm_joint: child link1_left -> left_link1
- joint right_arm_joint: child link1_right -> right_link1

File: ros2_ws/src/marvin/urdf/marvin.urdf.xacro (robot description, xacro)
@@ -38,5 +38,5 @@
   <joint name="left_arm_joint" type="fixed">
     <parent link="torso"/>
-    <child link="link1_left"/>
+    <child link="left_link1"/>
     <origin xyz="${left_arm_origin_xyz}" rpy="0 1.5708 0"/>
   </joint>
@@ -44,5 +44,5 @@
   <joint name="right_arm_joint" type="fixed">
     <parent link="torso"/>
-    <child link="link1_right"/>
+    <child link="right_link1"/>
     <origin xyz="${right_arm_origin_xyz}" rpy="0 1.5708 3.1415926535"/> <!-- Rotate by pi -->
   </joint>

File: ros2_ws/src/marvin_moveit/config/marvin.ros2_control.xacro (robot description, xacro)
@@ -8,71 +8,71 @@
                 <plugin>mock_components/GenericSystem</plugin>
             </hardware>
-            <joint name="gripper_left">
+            <joint name="left_gripper">
                 <command_interface name="position"/>
                 <state_interface name="position">
-                  <param name="initial_value">${initial_positions['gripper_left']}</param>
+                  <param name="initial_value">${initial_positions['left_gripper']}</param>
                 </state_interface>
                 <state_interface name="velocity"/>
             </joint>
-            <joint name="gripper_right">
+            <joint name="right_gripper">
                 <command_interface name="position"/>
                 <state_interface name="position">
-                  <param name="initial_value">${initial_positions['gripper_right']}</param>
+                  <param name="initial_value">${initial_positions['right_gripper']}</param>
                 </state_interface>
                 <state_interface name="velocity"/>
             </joint>
-            <joint name="joint1_right">
+            <joint name="right_joint1">
                 <command_interface name="position"/>
                 <state_interface name="position">
-                  <param name="initial_value">${initial_positions['joint1_right']}</param>
+                  <param name="initial_value">${initial_positions['right_joint1']}</param>
                 </state_interface>
                 <state_interface name="velocity"/>
             </joint>
-            <joint name="joint2_right">
+            <joint name="right_joint2">
                 <command_interface name="position"/>
                 <state_interface name="position">
-                  <param name="initial_value">${initial_positions['joint2_right']}</param>
+                  <param name="initial_value">${initial_positions['right_joint2']}</param>
                 </state_interface>
                 <state_interface name="velocity"/>
             </joint>
-            <joint name="joint3_right">
+            <joint name="right_joint3">
                 <command_interface name="position"/>
                 <state_interface name="position">
-                  <param name="initial_value">${initial_positions['joint3_right']}</param>
+                  <param name="initial_value">${initial_positions['right_joint3']}</param>
                 </state_interface>
                 <state_interface name="velocity"/>
             </joint>
-            <joint name="joint4_right">
+            <joint name="right_joint4">
                 <command_interface name="position"/>
                 <state_interface name="position">
-                  <param name="initial_value">${initial_positions['joint4_right']}</param>
+                  <param name="initial_value">${initial_positions['right_joint4']}</param>
                 </state_interface>
                 <state_interface name="velocity"/>
             </joint>
-            <joint name="joint1_left">
+            <joint name="left_joint1">
                 <command_interface name="position"/>
                 <state_interface name="position">
-                  <param name="initial_value">${initial_positions['joint1_left']}</param>
+                  <param name="initial_value">${initial_positions['left_joint1']}</param>
                 </state_interface>
                 <state_interface name="velocity"/>
             </joint>
-            <joint name="joint2_left">
+            <joint name="left_joint2">
                 <command_interface name="position"/>
                 <state_interface name="position">
-                  <param name="initial_value">${initial_positions['joint2_left']}</param>
+                  <param name="initial_value">${initial_positions['left_joint2']}</param>
                 </state_interface>
                 <state_interface name="velocity"/>
             </joint>
-            <joint name="joint3_left">
+            <joint name="left_joint3">
                 <command_interface name="position"/>
                 <state_interface name="position">
-                  <param name="initial_value">${initial_positions['joint3_left']}</param>
+                  <param name="initial_value">${initial_positions['left_joint3']}</param>
                 </state_interface>
                 <state_interface name="velocity"/>
             </joint>
-            <joint name="joint4_left">
+            <joint name="left_joint4">
                 <command_interface name="position"/>
                 <state_interface name="position">
-                  <param name="initial_value">${initial_positions['joint4_left']}</param>
+                  <param name="initial_value">${initial_positions['left_joint4']}</param>
                 </state_interface>
                 <state_interface name="velocity"/>

Commit message: urdf2 to urdf and custom_interfaces pkg bug fix

File: ros2_ws/src/marvin/urdf/marvin.urdf (robot description, URDF)
Before this commit: robot marvin, 18 links, 17 joints
Links:
- removed link left_end_effector_link
- removed link left_gripper_link
- removed link left_gripper_link_sub
- removed link left_link1
- removed link left_link2
- removed link left_link3
- removed link left_link4
- removed link left_link5
- removed link right_end_effector_link
- removed link right_gripper_link
- removed link right_gripper_link_sub
- removed link right_link1
- removed link right_link2
- removed link right_link3
- removed link right_link4
- removed link right_link5
- added link end_effector_link_left, mass 1.0e-03; visual box size=0.01 0.01 0.01
- added link end_effector_link_right, mass 1.0e-03; visual box size=0.01 0.01 0.01
- added link gripper_link_left, mass 1.0e-03; collision mesh filename=/home/jaeho/marvin/ros2_ws/install/marvin/share/marvin/mesh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 scale=0.001 0.001 0.001; visual mesh filename=/home/jaeho/marvin/ros2_ws/install/marvin/share/marvin/mesh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 scale=0.001 0.001 0.001
- added link gripper_link_right, mass 1.0e-03; collision mesh filename=/home/jaeho/marvin/ros2_ws/install/marvin/share/marvin/mesh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 scale=0.001 0.001 0.001; visual mesh filename=/home/jaeho/marvin/ros2_ws/install/marvin/share/marvin/mesh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 scale=0.001 0.001 0.001
- added link gripper_link_sub_left, mass 1.0e-03; collision mesh filename=/home/jaeho/marvin/ros2_ws/install/marvin/share/marvin/mesh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 scale=0.001 0.001 0.001; visual mesh filename=/home/jaeho/marvin/ros2_ws/install/marvin/share/marvin/mesh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 scale=0.001 0.001 0.001
- added link gripper_link_sub_right, mass 1.0e-03; collision mesh filename=/home/jaeho/marvin/ros2_ws/install/marvin/share/marvin/mesh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 scale=0.001 0.001 0.001; visual mesh filename=/home/jaeho/marvin/ros2_ws/install/marvin/share/marvin/mesh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 scale=0.001 0.001 0.001
- added link link1_left, mass 7.9119962e-02; collision mesh filename=/home/jaeho/marvin/ros2_ws/install/marvin/share/marvin/mesh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 scale=0.001 0.001 0.001; visual mesh filename=/home/jaeho/marvin/ros2_ws/install/marvin/share/marvin/mesh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 scale=0.001 0.001 0.001
- added link link1_right, mass 7.9119962e-02; collision mesh filename=/home/jaeho/marvin/ros2_ws/install/marvin/share/marvin/mesh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 scale=0.001 0.001 0.001; visual mesh filename=/home/jaeho/marvin/ros2_ws/install/marvin/share/marvin/mesh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 scale=0.001 0.001 0.001
- added link link2_left, mass 9.8406837e-02; collision mesh filename=/home/jaeho/marvin/ros2_ws/install/marvin/share/marvin/mesh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 scale=0.001 0.001 0.001; visual mesh filename=/home/jaeho/marvin/ros2_ws/install/marvin/share/marvin/mesh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 scale=0.001 0.001 0.001
- added link link2_right, mass 9.8406837e-02; collision mesh filename=/home/jaeho/marvin/ros2_ws/install/marvin/share/marvin/mesh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 scale=0.001 0.001 0.001; visual mesh filename=/home/jaeho/marvin/ros2_ws/install/marvin/share/marvin/mesh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 scale=0.001 0.001 0.001
- added link link3_left, mass 1.3850917e-01; collision mesh filename=/home/jaeho/marvin/ros2_ws/install/marvin/share/marvin/mesh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 scale=0.001 0.001 0.001; visual mesh filename=/home/jaeho/marvin/ros2_ws/install/marvin/share/marvin/mesh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 scale=0.001 0.001 0.001
- added link link3_right, mass 1.3850917e-01; collision mesh filename=/home/jaeho/marvin/ros2_ws/install/marvin/share/marvin/mesh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 scale=0.001 0.001 0.001; visual mesh filename=/home/jaeho/marvin/ros2_ws/install/marvin/share/marvin/mesh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 scale=0.001 0.001 0.001
- added link link4_left, mass 1.3274562e-01; collision mesh filename=/home/jaeho/marvin/ros2_ws/install/marvin/share/marvin/mesh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 scale=0.001 0.001 0.001; visual mesh filename=/home/jaeho/marvin/ros2_ws/install/marvin/share/marvin/mesh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 scale=0.001 0.001 0.001
- added link link4_right, mass 1.3274562e-01; collision mesh filename=/home/jaeho/marvin/ros2_ws/install/marvin/share/marvin/mesh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 scale=0.001 0.001 0.001; visual mesh filename=/home/jaeho/marvin/ros2_ws/install/marvin/share/marvin/mesh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 scale=0.001 0.001 0.001
- added link link5_left, mass 1.4327573e-01; collision mesh filename=/home/jaeho/marvin/ros2_ws/install/marvin/share/marvin/mesh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 scale=0.001 0.001 0.001; visual mesh filename=/home/jaeho/marvin/ros2_ws/install/marvin/share/marvin/mesh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 scale=0.001 0.001 0.001
- added link link5_right, mass 1.4327573e-01; collision mesh filename=/home/jaeho/marvin/ros2_ws/install/marvin/share/marvin/mesh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 scale=0.001 0.001 0.001; visual mesh filename=/home/jaeho/marvin/ros2_ws/install/marvin/share/marvin/mesh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 scale=0.001 0.001 0.001
Joints:
- removed joint left_end_effector_joint
- removed joint left_gripper
- removed joint left_gripper_sub
- removed joint left_joint1
- removed joint left_joint2
- removed joint left_joint3
- removed joint left_joint4
- removed joint right_end_effector_joint
- removed joint right_gripper
- removed joint right_gripper_sub
- removed joint right_joint1
- removed joint right_joint2
- removed joint right_joint3
- removed joint right_joint4
- added joint end_effector_joint_left: type fixed, parent link5_left, child end_effector_link_left, origin xyz=0.126 0.0 0.0 rpy=0 0 0
- added joint end_effector_joint_right: type fixed, parent link5_right, child end_effector_link_right, origin xyz=0.126 0.0 0.0 rpy=0 0 0
- added joint gripper_left: type prismatic, parent link5_left, child gripper_link_left, origin xyz=0.0817 0.021 0.0 rpy=0 0 0, axis 0 1 0, limit lower=-0.010 upper=0.019 effort=1 velocity=4.8
- added joint gripper_right: type prismatic, parent link5_right, child gripper_link_right, origin xyz=0.0817 0.021 0.0 rpy=0 0 0, axis 0 1 0, limit lower=-0.010 upper=0.019 effort=1 velocity=4.8
- added joint gripper_sub_left: type prismatic, parent link5_left, child gripper_link_sub_left, origin xyz=0.0817 -0.021 0 rpy=0 0 0, axis 0 -1 0, limit lower=-0.010 upper=0.019 effort=1 velocity=4.8, mimic joint=gripper_left multiplier=1
- added joint gripper_sub_right: type prismatic, parent link5_right, child gripper_link_sub_right, origin xyz=0.0817 -0.021 0 rpy=0 0 0, axis 0 -1 0, limit lower=-0.010 upper=0.019 effort=1 velocity=4.8, mimic joint=gripper_right multiplier=1
- added joint joint1_left: type revolute, parent link1_left, child link2_left, origin xyz=0.012 0.0 0.017 rpy=0 0 0, axis 0 0 1, limit lower=-2.827433388230814 upper=2.827433388230814 effort=1 velocity=4.8
- added joint joint1_right: type revolute, parent link1_right, child link2_right, origin xyz=0.012 0.0 0.017 rpy=0 0 0, axis 0 0 1, limit lower=-2.827433388230814 upper=2.827433388230814 effort=1 velocity=4.8
- added joint joint2_left: type revolute, parent link2_left, child link3_left, origin xyz=0.0 0.0 0.0595 rpy=0 0 0, axis 0 1 0, limit lower=-1.790707812546182 upper=1.5707963267948966 effort=1 velocity=4.8
- added joint joint2_right: type revolute, parent link2_right, child link3_right, origin xyz=0.0 0.0 0.0595 rpy=0 0 0, axis 0 1 0, limit lower=-1.790707812546182 upper=1.5707963267948966 effort=1 velocity=4.8
- added joint joint3_left: type revolute, parent link3_left, child link4_left, origin xyz=0.024 0 0.128 rpy=0 0 0, axis 0 1 0, limit lower=-0.9424777960769379 upper=1.382300767579509 effort=1 velocity=4.8
- added joint joint3_right: type revolute, parent link3_right, child link4_right, origin xyz=0.024 0 0.128 rpy=0 0 0, axis 0 1 0, limit lower=-0.9424777960769379 upper=1.382300767579509 effort=1 velocity=4.8
- added joint joint4_left: type revolute, parent link4_left, child link5_left, origin xyz=0.124 0.0 0.0 rpy=0 0 0, axis 0 1 0, limit lower=-1.790707812546182 upper=2.0420352248333655 effort=1 velocity=4.8
- added joint joint4_right: type revolute, parent link4_right, child link5_right, origin xyz=0.124 0.0 0.0 rpy=0 0 0, axis 0 1 0, limit lower=-1.790707812546182 upper=2.0420352248333655 effort=1 velocity=4.8

File: ros2_ws/src/marvin/urdf/marvin.urdf.xacro (robot description, xacro)
@@ -3,12 +3,12 @@
 <robot name="marvin" xmlns:xacro="http://ros.org/wiki/xacro">
   <!-- Import Rviz colors -->
-  <xacro:include filename="/home/jaeho/marvin/ros2_ws/src/marvin/urdf2/materials.xacro" />
+  <xacro:include filename="/home/jaeho/marvin/ros2_ws/src/marvin/urdf/materials.xacro" />
   <!-- Import all Gazebo-customization elements, including Gazebo colors -->
-  <!--xacro:include filename="/home/jaeho/marvin/ros2_ws/src/marvin/urdf2/open_manipulator.gazebo.xacro" /-->
+  <!--xacro:include filename="/home/jaeho/marvin/ros2_ws/src/marvin/urdf/open_manipulator.gazebo.xacro" /-->
   <!-- Import Transmission -->
-  <xacro:include filename="/home/jaeho/marvin/ros2_ws/src/marvin/urdf2/open_manipulator.transmission.xacro" />
+  <xacro:include filename="/home/jaeho/marvin/ros2_ws/src/marvin/urdf/open_manipulator.transmission.xacro" />
   <!-- Import URDF -->
-  <!--xacro:include filename="/home/jaeho/marvin/ros2_ws/src/marvin/urdf2/open_manipulator.urdf.xacro" /-->
-  <xacro:include filename="/home/jaeho/marvin/ros2_ws/src/marvin/urdf2/single_arm.xacro" />
+  <!--xacro:include filename="/home/jaeho/marvin/ros2_ws/src/marvin/urdf/open_manipulator.urdf.xacro" /-->
+  <xacro:include filename="/home/jaeho/marvin/ros2_ws/src/marvin/urdf/single_arm.xacro" />
   <!-- World -->
   <link name="world"/>
