Commit message: hardware bringup

File: ros2_ws/src/marvin/urdf/marvin.urdf.xacro (robot description, xacro)
@@ -3,12 +3,12 @@
 <robot name="marvin" xmlns:xacro="http://ros.org/wiki/xacro">
   <!-- Import Rviz colors -->
-  <xacro:include filename="/home/jaeho/marvin/ros2_ws/src/marvin/urdf2/materials.xacro" />
+  <xacro:include filename="$(find marvin)/urdf/materials.xacro" />
   <!-- Import all Gazebo-customization elements, including Gazebo colors -->
   <!--xacro:include filename="/home/jaeho/marvin/ros2_ws/src/marvin/urdf2/open_manipulator.gazebo.xacro" /-->
   <!-- Import Transmission -->
-  <xacro:include filename="/home/jaeho/marvin/ros2_ws/src/marvin/urdf2/open_manipulator.transmission.xacro" />
+  <!-- xacro:include filename="$(find marvin)/urdf/open_manipulator.transmission.xacro" /-->
   <!-- Import URDF -->
   <!--xacro:include filename="/home/jaeho/marvin/ros2_ws/src/marvin/urdf2/open_manipulator.urdf.xacro" /-->
-  <xacro:include filename="/home/jaeho/marvin/ros2_ws/src/marvin/urdf2/single_arm.xacro" />
+  <xacro:include filename="$(find marvin)/urdf/single_arm.xacro" />
   <!-- World -->
   <link name="world"/>

File: ros2_ws/src/marvin/urdf/single_arm.xacro (robot description, xacro)
@@ -3,5 +3,5 @@
   <xacro:macro name="arm" params="name">
     <!-- Link 1 -->
-    <link name="link1_${name}">
+    <link name="${name}_link1">
       <visual>
         <origin xyz="0 0 0" rpy="0 0 0"/>
@@ -27,7 +27,7 @@
     </link>
     <!-- Joint 1 -->
-    <joint name="joint1_${name}" type="revolute">
-      <parent link="link1_${name}"/>
-      <child link="link2_${name}"/>
+    <joint name="${name}_joint1" type="revolute">
+      <parent link="${name}_link1"/>
+      <child link="${name}_link2"/>
       <origin xyz="0.012 0.0 0.017" rpy="0 0 0"/>
       <axis xyz="0 0 1"/>
@@ -35,5 +35,5 @@
     </joint>
     <!--  Link 2 -->
-    <link name="link2_${name}">
+    <link name="${name}_link2">
       <visual>
         <origin xyz="0 0 0.019" rpy="0 0 0"/>
@@ -58,7 +58,7 @@
     </link>
     <!--  Joint 2 -->
-    <joint name="joint2_${name}" type="revolute">
-      <parent link="link2_${name}"/>
-      <child link="link3_${name}"/>
+    <joint name="${name}_joint2" type="revolute">
+      <parent link="${name}_link2"/>
+      <child link="${name}_link3"/>
       <origin xyz="0.0 0.0 0.0595" rpy="0 0 0"/>
       <axis xyz="0 1 0"/>
@@ -66,5 +66,5 @@
     </joint>
     <!--  Link 3 -->
-    <link name="link3_${name}">
+    <link name="${name}_link3">
       <visual>
         <origin xyz="0 0 0" rpy="0 0 0"/>
@@ -89,7 +89,7 @@
     </link>
     <!--  Joint 3 -->
-    <joint name="joint3_${name}" type="revolute">
-      <parent link="link3_${name}"/>
-      <child link="link4_${name}"/>
+    <joint name="${name}_joint3" type="revolute">
+      <parent link="${name}_link3"/>
+      <child link="${name}_link4"/>
       <origin xyz="0.024 0 0.128" rpy="0 0 0"/>
       <axis xyz="0 1 0"/>
@@ -97,5 +97,5 @@
     </joint>
     <!--  Link 4 -->
-    <link name="link4_${name}">
+    <link name="${name}_link4">
       <visual>
         <origin xyz="0 0 0" rpy="0 0 0"/>
@@ -120,7 +120,7 @@
     </link>
     <!--  Joint 4 -->
-    <joint name="joint4_${name}" type="revolute">
-      <parent link="link4_${name}"/>
-      <child link="link5_${name}"/>
+    <joint name="${name}_joint4" type="revolute">
+      <parent link="${name}_link4"/>
+      <child link="${name}_link5"/>
       <origin xyz="0.124 0.0 0.0" rpy="0 0 0"/>
       <axis xyz="0 1 0"/>
@@ -128,5 +128,5 @@
     </joint>
     <!--  Link 5 -->
-    <link name="link5_${name}">
+    <link name="${name}_link5">
       <visual>
         <origin xyz="0 0 0" rpy="0 0 0"/>
@@ -151,7 +151,7 @@
     </link>
     <!--  Gripper joint -->
-    <joint name="gripper_${name}" type="prismatic">
-      <parent link="link5_${name}"/>
-      <child link="gripper_link_${name}"/>
+    <joint name="${name}_gripper" type="prismatic">
+      <parent link="${name}_link5"/>
+      <child link="${name}_gripper_link"/>
       <origin xyz="0.0817 0.021 0.0" rpy="0 0 0"/>
       <axis xyz="0 1 0"/>
@@ -159,5 +159,5 @@
     </joint>
     <!--  Gripper link -->
-    <link name="gripper_link_${name}">
+    <link name="${name}_gripper_link">
       <visual>
         <origin xyz="0.0 0.0 0" rpy="0 0 0"/>
@@ -182,14 +182,14 @@
     </link>
     <!--  Gripper joint sub -->
-    <joint name="gripper_sub_${name}" type="prismatic">
-      <parent link="link5_${name}"/>
-      <child link="gripper_link_sub_${name}"/>
+    <joint name="${name}_gripper_sub" type="prismatic">
+      <parent link="${name}_link5"/>
+      <child link="${name}_gripper_link_sub"/>
       <origin xyz="0.0817 -0.021 0" rpy="0 0 0"/>
       <axis xyz="0 -1 0"/>
       <limit velocity="4.8" effort="1" lower="-0.010" upper="0.019" />
-      <mimic joint="gripper_${name}" multiplier="1"/>
+      <mimic joint="${name}_gripper" multiplier="1"/>
     </joint>
     <!--  Gripper link sub -->
-    <link name="gripper_link_sub_${name}">
+    <link name="${name}_gripper_link_sub">
       <visual>
         <origin xyz="0.0 -0.0 0" rpy="0 0 0"/>
@@ -214,11 +214,11 @@
     </link>
     <!-- end effector joint -->
-    <joint name="end_effector_joint_${name}" type="fixed">
+    <joint name="${name}_end_effector_joint" type="fixed">
       <origin xyz="0.126 0.0 0.0" rpy="0 0 0"/>
-      <parent link="link5_${name}"/>
-      <child link="end_effector_link_${name}"/>
+      <parent link="${name}_link5"/>
+      <child link="${name}_end_effector_link"/>
     </joint>
     <!-- end effector link -->
-    <link name="end_effector_link_${name}">
+    <link name="${name}_end_effector_link">
       <visual>
         <origin xyz="0 0 0" rpy="0 0 0"/>
