Commit message: blah

File: ros2_ws/src/marvin/urdf/single_arm.xacro (robot description, xacro)
@@ -7,12 +7,12 @@
         <origin xyz="0 0 0" rpy="0 0 0"/>
         <geometry>
-          <mesh filename="package://meshes/stl/chain_link1.stl" scale="0.001 0.001 0.001"/>
-        </geometry>
-        <material name="grey"/>
-      </visual>
-      <collision>
-        <origin xyz="0 0 0" rpy="0 0 0"/>
-        <geometry>
-          <mesh filename="package://meshes/stl/chain_link1.stl" scale="0.001 0.001 0.001"/>
+          <mesh filename="package://marvin/meshes/stl/chain_link1.stl" scale="0.001 0.001 0.001"/>
+        </geometry>
+        <material name="grey"/>
+      </visual>
+      <collision>
+        <origin xyz="0 0 0" rpy="0 0 0"/>
+        <geometry>
+          <mesh filename="package://marvin/meshes/stl/chain_link1.stl" scale="0.001 0.001 0.001"/>
         </geometry>
       </collision>
@@ -39,5 +39,5 @@
         <origin xyz="0 0 0.019" rpy="0 0 0"/>
         <geometry>
-          <mesh filename="package://meshes/stl/chain_link2.stl" scale="0.001 0.001 0.001"/>
+          <mesh filename="package://marvin/meshes/stl/chain_link2.stl" scale="0.001 0.001 0.001"/>
         </geometry>
         <material name="grey"/>
@@ -46,5 +46,5 @@
         <origin xyz="0 0 0.019" rpy="0 0 0"/>
         <geometry>
-          <mesh filename="package://meshes/stl/chain_link2.stl" scale="0.001 0.001 0.001"/>
+          <mesh filename="package://marvin/meshes/stl/chain_link2.stl" scale="0.001 0.001 0.001"/>
         </geometry>
       </collision>
@@ -70,12 +70,12 @@
         <origin xyz="0 0 0" rpy="0 0 0"/>
         <geometry>
-          <mesh filename="package://meshes/stl/chain_link3.stl" scale="0.001 0.001 0.001"/>
-        </geometry>
-        <material name="grey"/>
-      </visual>
-      <collision>
-        <origin xyz="0 0 0" rpy="0 0 0"/>
-        <geometry>
-          <mesh filename="package://meshes/stl/chain_link3.stl" scale="0.001 0.001 0.001"/>
+          <mesh filename="package://marvin/meshes/stl/chain_link3.stl" scale="0.001 0.001 0.001"/>
+        </geometry>
+        <material name="grey"/>
+      </visual>
+      <collision>
+        <origin xyz="0 0 0" rpy="0 0 0"/>
+        <geometry>
+          <mesh filename="package://marvin/meshes/stl/chain_link3.stl" scale="0.001 0.001 0.001"/>
         </geometry>
       </collision>
@@ -101,12 +101,12 @@
         <origin xyz="0 0 0" rpy="0 0 0"/>
         <geometry>
-          <mesh filename="package://meshes/stl/chain_link4.stl" scale="0.001 0.001 0.001"/>
-        </geometry>
-        <material name="grey"/>
-      </visual>
-      <collision>
-        <origin xyz="0 0 0" rpy="0 0 0"/>
-        <geometry>
-          <mesh filename="package://meshes/stl/chain_link4.stl" scale="0.001 0.001 0.001"/>
+          <mesh filename="package://marvin/meshes/stl/chain_link4.stl" scale="0.001 0.001 0.001"/>
+        </geometry>
+        <material name="grey"/>
+      </visual>
+      <collision>
+        <origin xyz="0 0 0" rpy="0 0 0"/>
+        <geometry>
+          <mesh filename="package://marvin/meshes/stl/chain_link4.stl" scale="0.001 0.001 0.001"/>
         </geometry>
       </collision>
@@ -132,12 +132,12 @@
         <origin xyz="0 0 0" rpy="0 0 0"/>
         <geometry>
-          <mesh filename="package://meshes/stl/chain_link5.stl" scale="0.001 0.001 0.001"/>
-        </geometry>
-        <material name="grey"/>
-      </visual>
-      <collision>
-        <origin xyz="0 0 0" rpy="0 0 0"/>
-        <geometry>
-          <mesh filename="package://meshes/stl/chain_link5.stl" scale="0.001 0.001 0.001"/>
+          <mesh filename="package://marvin/meshes/stl/chain_link5.stl" scale="0.001 0.001 0.001"/>
+        </geometry>
+        <material name="grey"/>
+      </visual>
+      <collision>
+        <origin xyz="0 0 0" rpy="0 0 0"/>
+        <geometry>
+          <mesh filename="package://marvin/meshes/stl/chain_link5.stl" scale="0.001 0.001 0.001"/>
         </geometry>
       </collision>
@@ -163,5 +163,5 @@
         <origin xyz="0.0 0.0 0" rpy="0 0 0"/>
         <geometry>
-          <mesh filename="package://meshes/stl/chain_link_grip_l.stl" scale="0.001 0.001 0.001"/>
+          <mesh filename="package://marvin/meshes/stl/chain_link_grip_l.stl" scale="0.001 0.001 0.001"/>
         </geometry>
         <material name="grey"/>
@@ -170,5 +170,5 @@
         <origin xyz="0.0 0.0 0" rpy="0 0 0"/>
         <geometry>
-          <mesh filename="package://meshes/stl/chain_link_grip_l.stl" scale="0.001 0.001 0.001"/>
+          <mesh filename="package://marvin/meshes/stl/chain_link_grip_l.stl" scale="0.001 0.001 0.001"/>
         </geometry>
       </collision>
@@ -195,5 +195,5 @@
         <origin xyz="0.0 -0.0 0" rpy="0 0 0"/>
         <geometry>
-          <mesh filename="package://meshes/stl/chain_link_grip_r.stl" scale="0.001 0.001 0.001"/>
+          <mesh filename="package://marvin/meshes/stl/chain_link_grip_r.stl" scale="0.001 0.001 0.001"/>
         </geometry>
         <material name="grey"/>
@@ -202,5 +202,5 @@
         <origin xyz="0.0 -0.0 0" rpy="0 0 0"/>
         <geometry>
-          <mesh filename="package://meshes/stl/chain_link_grip_r.stl" scale="0.001 0.001 0.001"/>
+          <mesh filename="package://marvin/meshes/stl/chain_link_grip_r.stl" scale="0.001 0.001 0.001"/>
         </geometry>
       </collision>
@@ -228,4 +228,11 @@
         <material name="red"/>
       </visual>
+      <collision>
+        <origin xyz="0 0 0" rpy="0 0 0"/>
+        <geometry>
+          <box size="0.01 0.01 0.01" />
+        </geometry>
+        <material name="red"/>
+      </collision>
       <inertial>
         <origin xyz="0 0 0" />
