Commit message: fix urdf
clean blender

rviz

File: blender/exports/marvin/urdf/marvin.urdf (robot description, URDF)
Before this commit: robot marvin, 15 links, 14 joints
Links:
- link left_gripper_link: geometry collision mesh filename=package://marvin/meshes/stl/chain_link_grip_l.stl scale=0.00100 0.00100 0.00100; visual mesh filename=package://marvin/meshes/stl/chain_link_grip_l.stl scale=0.00100 0.00100 0.00100
- link left_gripper_link_sub: geometry collision mesh filename=package://marvin/meshes/stl/chain_link_grip_r.stl scale=0.00100 0.00100 0.00100; visual mesh filename=package://marvin/meshes/stl/chain_link_grip_r.stl scale=0.00100 0.00100 0.00100
- link left_link2: geometry collision mesh filename=package://marvin/meshes/stl/chain_link2.stl scale=0.00100 0.00100 0.00100; visual mesh filename=package://marvin/meshes/stl/chain_link2.stl scale=0.00100 0.00100 0.00100
- link left_link3: geometry collision mesh filename=package://marvin/meshes/stl/chain_link3.stl scale=0.00100 0.00100 0.00100; visual mesh filename=package://marvin/meshes/stl/chain_link3.stl scale=0.00100 0.00100 0.00100
- link left_link4: geometry collision mesh filename=package://marvin/meshes/stl/chain_link4.stl scale=0.00100 0.00100 0.00100; visual mesh filename=package://marvin/meshes/stl/chain_link4.stl scale=0.00100 0.00100 0.00100
- link left_link5: geometry collision mesh filename=package://marvin/meshes/stl/chain_link5.stl scale=0.00100 0.00100 0.00100; visual mesh filename=package://marvin/meshes/stl/chain_link5.stl scale=0.00100 0.00100 0.00100
- link marvin: geometry collision mesh filename=package://marvin/meshes/stl/chain_link1.stl scale=0.00100 0.00100 0.00100; collision mesh filename=package://marvin/meshes/stl/chain_link1.stl scale=0.00100 0.00100 0.00100
- link right_gripper_link: geometry collision mesh filename=package://marvin/meshes/stl/chain_link_grip_l.stl scale=0.00100 0.00100 0.00100; visual mesh filename=package://marvin/meshes/stl/chain_link_grip_l.stl scale=0.00100 0.00100 0.00100
- link right_gripper_link_sub: geometry collision mesh filename=package://marvin/meshes/stl/chain_link_grip_r.stl scale=0.00100 0.00100 0.00100; visual mesh filename=package://marvin/meshes/stl/chain_link_grip_r.stl scale=0.00100 0.00100 0.00100
- link right_link2: geometry collision mesh filename=package://marvin/meshes/stl/chain_link2.stl scale=0.00100 0.00100 0.00100; visual mesh filename=package://marvin/meshes/stl/chain_link2.stl scale=0.00100 0.00100 0.00100
- link right_link3: geometry collision mesh filename=package://marvin/meshes/stl/chain_link3.stl scale=0.00100 0.00100 0.00100; visual mesh filename=package://marvin/meshes/stl/chain_link3.stl scale=0.00100 0.00100 0.00100
- link right_link4: geometry collision mesh filename=package://marvin/meshes/stl/chain_link4.stl scale=0.00100 0.00100 0.00100; visual mesh filename=package://marvin/meshes/stl/chain_link4.stl scale=0.00100 0.00100 0.00100
- link right_link5: geometry collision mesh filename=package://marvin/meshes/stl/chain_link5.stl scale=0.00100 0.00100 0.00100; visual mesh filename=package://marvin/meshes/stl/chain_link5.stl scale=0.00100 0.00100 0.00100
Joints:
- joint right_gripper_sub: mimic joint=left_gripper multiplier=1.00000 offset=0.00000 -> joint=right_gripper multiplier=1.00000 offset=0.00000
- joint right_joint1: origin xyz=0.09700 0.00000 -0.01200 rpy=-0.00000 1.57080 -0.00000 -> xyz=0.09700 -0.00000 -0.01200 rpy=-0.00000 1.57080 -0.00000

File: ros2_ws/src/marvin/urdf/marvin.urdf (robot description, URDF)
Before this commit: robot marvin, 16 links, 15 joints
Links:
- removed link marvin_fixed_frame
- added link world
- link marvin: geometry collision mesh filename=package://marvin/meshes/stl/chain_link1.stl scale=0.00100 0.00100 0.00100; collision mesh filename=package://marvin/meshes/stl/chain_link1.stl scale=0.00100 0.00100 0.00100
- link right_gripper_link: geometry collision mesh filename=package://marvin/meshes/stl/chain_link_grip_l.stl scale=0.00100 0.00100 0.00100; visual mesh filename=package://marvin/meshes/stl/chain_link_grip_l.stl scale=0.00100 0.00100 0.00100
- link right_gripper_link_sub: geometry collision mesh filename=package://marvin/meshes/stl/chain_link_grip_r.stl scale=0.00100 0.00100 0.00100; visual mesh filename=package://marvin/meshes/stl/chain_link_grip_r.stl scale=0.00100 0.00100 0.00100
- link right_link2: geometry collision mesh filename=package://marvin/meshes/stl/chain_link2.stl scale=0.00100 0.00100 0.00100; visual mesh filename=package://marvin/meshes/stl/chain_link2.stl scale=0.00100 0.00100 0.00100
- link right_link3: geometry collision mesh filename=package://marvin/meshes/stl/chain_link3.stl scale=0.00100 0.00100 0.00100; visual mesh filename=package://marvin/meshes/stl/chain_link3.stl scale=0.00100 0.00100 0.00100
- link right_link4: geometry collision mesh filename=package://marvin/meshes/stl/chain_link4.stl scale=0.00100 0.00100 0.00100; visual mesh filename=package://marvin/meshes/stl/chain_link4.stl scale=0.00100 0.00100 0.00100
- link right_link5: geometry collision mesh filename=package://marvin/meshes/stl/chain_link5.stl scale=0.00100 0.00100 0.00100; visual mesh filename=package://marvin/meshes/stl/chain_link5.stl scale=0.00100 0.00100 0.00100
Joints:
- joint base_joint: parent marvin_fixed_frame -> world
- joint right_joint1: origin xyz=0.09700 0.00000 -0.01200 rpy=-0.00000 1.57080 -0.00000 -> xyz=0.09700 -0.00000 -0.01200 rpy=-0.00000 1.57080 -0.00000
