Commit message: hardware launch

File: ros2_ws/src/marvin/ros2_control/open_manipulator_x_system.ros2_control.xacro (robot description, xacro)
@@ -37,5 +37,7 @@
             <param name="port_name">${port_name}</param>
             <param name="baud_rate">1000000</param>
-            <param name="error_timeout_sec">0.2</param>
+            <!--param name="error_timeout_sec">0.2</param-->
+            <param name="error_timeout_ms">200</param>  <!-- 0.2 s -->
+            <param name="torque_enable">1</param>
             <param name="dynamixel_model_folder">/param/dxl_model</param>
             <!-- 4 revolute + 1 actuated gripper = 5 transmissions; 6th joint is the mimic -->
@@ -59,5 +61,5 @@
               0, 0, 0, 0, 1, 0
             </param>
-            <param name="ros_update_freq">200</param>
+            <param name="ros_update_freq">100</param>
             <param name="dynamixel_state_pub_msg_name">dynamixel_hardware_interface/dxl_state</param>
             <param name="get_dynamixel_data_srv_name">dynamixel_hardware_interface/get_dxl_data</param>
@@ -119,5 +121,5 @@
       </joint>
       <!-- Dynamixel devices on this port -->
-      <gpio name="dxl1">
+      <gpio name="${side}_dxl1">
         <param name="type">dxl</param>
         <param name="ID">${dxl_id1}</param>
@@ -136,5 +138,5 @@
         <param name="Return Delay Time">0</param>
       </gpio>
-      <gpio name="dxl2">
+      <gpio name="${side}_dxl2">
         <param name="type">dxl</param>
         <param name="ID">${dxl_id2}</param>
@@ -153,5 +155,5 @@
         <param name="Return Delay Time">0</param>
       </gpio>
-      <gpio name="dxl3">
+      <gpio name="${side}_dxl3">
         <param name="type">dxl</param>
         <param name="ID">${dxl_id3}</param>
@@ -170,5 +172,5 @@
         <param name="Return Delay Time">0</param>
       </gpio>
-      <gpio name="dxl4">
+      <gpio name="${side}_dxl4">
         <param name="type">dxl</param>
         <param name="ID">${dxl_id4}</param>
@@ -187,5 +189,5 @@
         <param name="Return Delay Time">0</param>
       </gpio>
-      <gpio name="dxl5">
+      <gpio name="${side}_dxl5">
         <param name="type">dxl</param>
         <param name="ID">${dxl_id5}</param>

File: ros2_ws/src/marvin/urdf/marvin_robot.urdf.xacro (robot description, xacro)
@@ -7,6 +7,6 @@
   <xacro:arg name="use_fake_hardware" default="false" />
   <xacro:arg name="fake_sensor_commands" default="false" />
-  <xacro:arg name="port_name_left" default="/dev/ttyUSB0" />
-  <xacro:arg name="port_name_right" default="/dev/ttyUSB1" />
+  <xacro:arg name="port_name_left" default="/dev/ttyUSB1" />
+  <xacro:arg name="port_name_right" default="/dev/ttyUSB0" />
   <!-- Import Rviz colors -->
   <xacro:include filename="$(find marvin)/urdf/materials.xacro" />
@@ -62,5 +62,5 @@
   <xacro:open_manipulator_x_gazebo side="right" />
   <xacro:open_manipulator_x_system
-    name="OpenManipulatorXSystem" prefix="$(arg prefix)"
+    name="left_arm_system" prefix="$(arg prefix)"
     side ="left"
     use_sim="$(arg use_sim)"
@@ -69,5 +69,5 @@
     port_name="$(arg port_name_left)"/>
     <xacro:open_manipulator_x_system
-    name="OpenManipulatorXSystem" prefix="$(arg prefix)"
+    name="right_arm_system" prefix="$(arg prefix)"
     side ="right"
     use_sim="$(arg use_sim)"

File: ros2_ws/src/marvin/urdf/single_arm.xacro (robot description, xacro)
@@ -7,12 +7,12 @@
         <origin xyz="0 0 0" rpy="0 0 0"/>
         <geometry>
-          <mesh filename="$(find marvin)/meshes/stl/chain_link1.stl" scale="0.001 0.001 0.001"/>
-        </geometry>
-        <material name="grey"/>
-      </visual>
-      <collision>
-        <origin xyz="0 0 0" rpy="0 0 0"/>
-        <geometry>
-          <mesh filename="$(find marvin)/meshes/stl/chain_link1.stl" scale="0.001 0.001 0.001"/>
+          <mesh filename="package://meshes/stl/chain_link1.stl" scale="0.001 0.001 0.001"/>
+        </geometry>
+        <material name="grey"/>
+      </visual>
+      <collision>
+        <origin xyz="0 0 0" rpy="0 0 0"/>
+        <geometry>
+          <mesh filename="package://meshes/stl/chain_link1.stl" scale="0.001 0.001 0.001"/>
         </geometry>
       </collision>
@@ -39,5 +39,5 @@
         <origin xyz="0 0 0.019" rpy="0 0 0"/>
         <geometry>
-          <mesh filename="$(find marvin)/meshes/stl/chain_link2.stl" scale="0.001 0.001 0.001"/>
+          <mesh filename="package://meshes/stl/chain_link2.stl" scale="0.001 0.001 0.001"/>
         </geometry>
         <material name="grey"/>
@@ -46,5 +46,5 @@
         <origin xyz="0 0 0.019" rpy="0 0 0"/>
         <geometry>
-          <mesh filename="$(find marvin)/meshes/stl/chain_link2.stl" scale="0.001 0.001 0.001"/>
+          <mesh filename="package://meshes/stl/chain_link2.stl" scale="0.001 0.001 0.001"/>
         </geometry>
       </collision>
@@ -70,12 +70,12 @@
         <origin xyz="0 0 0" rpy="0 0 0"/>
         <geometry>
-          <mesh filename="$(find marvin)/meshes/stl/chain_link3.stl" scale="0.001 0.001 0.001"/>
-        </geometry>
-        <material name="grey"/>
-      </visual>
-      <collision>
-        <origin xyz="0 0 0" rpy="0 0 0"/>
-        <geometry>
-          <mesh filename="$(find marvin)/meshes/stl/chain_link3.stl" scale="0.001 0.001 0.001"/>
+          <mesh filename="package://meshes/stl/chain_link3.stl" scale="0.001 0.001 0.001"/>
+        </geometry>
+        <material name="grey"/>
+      </visual>
+      <collision>
+        <origin xyz="0 0 0" rpy="0 0 0"/>
+        <geometry>
+          <mesh filename="package://meshes/stl/chain_link3.stl" scale="0.001 0.001 0.001"/>
         </geometry>
       </collision>
@@ -101,12 +101,12 @@
         <origin xyz="0 0 0" rpy="0 0 0"/>
         <geometry>
-          <mesh filename="$(find marvin)/meshes/stl/chain_link4.stl" scale="0.001 0.001 0.001"/>
-        </geometry>
-        <material name="grey"/>
-      </visual>
-      <collision>
-        <origin xyz="0 0 0" rpy="0 0 0"/>
-        <geometry>
-          <mesh filename="$(find marvin)/meshes/stl/chain_link4.stl" scale="0.001 0.001 0.001"/>
+          <mesh filename="package://meshes/stl/chain_link4.stl" scale="0.001 0.001 0.001"/>
+        </geometry>
+        <material name="grey"/>
+      </visual>
+      <collision>
+        <origin xyz="0 0 0" rpy="0 0 0"/>
+        <geometry>
+          <mesh filename="package://meshes/stl/chain_link4.stl" scale="0.001 0.001 0.001"/>
         </geometry>
       </collision>
@@ -132,12 +132,12 @@
         <origin xyz="0 0 0" rpy="0 0 0"/>
         <geometry>
-          <mesh filename="$(find marvin)/meshes/stl/chain_link5.stl" scale="0.001 0.001 0.001"/>
-        </geometry>
-        <material name="grey"/>
-      </visual>
-      <collision>
-        <origin xyz="0 0 0" rpy="0 0 0"/>
-        <geometry>
-          <mesh filename="$(find marvin)/meshes/stl/chain_link5.stl" scale="0.001 0.001 0.001"/>
+          <mesh filename="package://meshes/stl/chain_link5.stl" scale="0.001 0.001 0.001"/>
+        </geometry>
+        <material name="grey"/>
+      </visual>
+      <collision>
+        <origin xyz="0 0 0" rpy="0 0 0"/>
+        <geometry>
+          <mesh filename="package://meshes/stl/chain_link5.stl" scale="0.001 0.001 0.001"/>
         </geometry>
       </collision>
@@ -163,5 +163,5 @@
         <origin xyz="0.0 0.0 0" rpy="0 0 0"/>
         <geometry>
-          <mesh filename="$(find marvin)/meshes/stl/chain_link_grip_l.stl" scale="0.001 0.001 0.001"/>
+          <mesh filename="package://meshes/stl/chain_link_grip_l.stl" scale="0.001 0.001 0.001"/>
         </geometry>
         <material name="grey"/>
@@ -170,5 +170,5 @@
         <origin xyz="0.0 0.0 0" rpy="0 0 0"/>
         <geometry>
-          <mesh filename="$(find marvin)/meshes/stl/chain_link_grip_l.stl" scale="0.001 0.001 0.001"/>
+          <mesh filename="package://meshes/stl/chain_link_grip_l.stl" scale="0.001 0.001 0.001"/>
         </geometry>
       </collision>
@@ -195,5 +195,5 @@
         <origin xyz="0.0 -0.0 0" rpy="0 0 0"/>
         <geometry>
-          <mesh filename="$(find marvin)/meshes/stl/chain_link_grip_r.stl" scale="0.001 0.001 0.001"/>
+          <mesh filename="package://meshes/stl/chain_link_grip_r.stl" scale="0.001 0.001 0.001"/>
         </geometry>
         <material name="grey"/>
@@ -202,5 +202,5 @@
         <origin xyz="0.0 -0.0 0" rpy="0 0 0"/>
         <geometry>
-          <mesh filename="$(find marvin)/meshes/stl/chain_link_grip_r.stl" scale="0.001 0.001 0.001"/>
+          <mesh filename="package://meshes/stl/chain_link_grip_r.stl" scale="0.001 0.001 0.001"/>
         </geometry>
       </collision>
